File: led.sch (EAGLE design)
At the start: 4 parts

Commit message: save
Parts:
- removed U$1, U$2, U$3, U$4: TPS92513TPS92513HV, derek:TPS92513TPS92513HV
- added C1: Value, derek:GRM32ER71J106KA12L
- added C2: GCM155R71H103KA55D, derek:GCM155R71H103KA55D
- added C3: CC0805KRX7R9BB103, derek:CC0805KRX7R9BB103
- added C4: CC0805KRX7R8BB104, derek:CC0805KRX7R8BB104
- added C5: 08053C104KAT2A, derek:08053C104KAT2A
- added C6: GMK212B7105KG-T, derek:GMK212B7105KG-T
- added D1: BAT54WSTR, derek:BAT54WSTR
- added D2: PMEG6010CEH,115, derek:PMEG6010CEH,115
- added L1: 74408943220, derek:74408943220
- added R1: CRCW0402121KFKED, derek:CRCW0402121KFKED
- added R2: CRCW04027K68FKED, derek:CRCW04027K68FKED
- added R3, R5: CRCW04021K00FKED, derek:CRCW04021K00FKED
- added R4: CRCW0402162KFKED, derek:CRCW0402162KFKED
- added R6: CRM0805-FX-R510ELF, derek:CRM0805-FX-R510ELF
- added U1: TPS92513HV, derek:TPS92513HV
Connections:
- new net N$1: C1.2, C2.2, C3.2, C4.2, D1.A, R2.2, R3.2, R4.2, R6.2, U1.GND
- new net N$10: C5.2, U1.BOOT
- new net N$11: R5.2, U1.ISENSE
- new net N$2: C3.1, R3.1, U1.IADJ
- new net N$3: R1.2, R2.1, U1.UVLO
- new net N$4: C1.1, C2.1, D2.K, R1.1, U1.VIN
- new net N$5: C5.1, D1.K, L1.1, U1.PH
- new net N$6: C6.2, R5.1, R6.1
- new net N$7: C6.1, D2.A, L1.2
- new net N$8: R4.1, U1.RT/CLK
- new net N$9: C4.1, U1.COMP

Commit message: save
Parts:
- added D3, D4, D5, D6, D7: XPGWHT, derek:XPGWHT
- added J1: (no value), derek:CONN_02
- C1: value Value -> GRM32ER71J106KA12L
Connections:
- removed net N$1: C1.2, C2.2, C3.2, C4.2, D1.A, R2.2, R3.2, R4.2, R6.2, U1.GND
- new net GND: C1.2, C2.2, C3.2, C4.2, D1.A, J1.1, R2.2, R3.2, R4.2, R6.2, U1.GND
- new net N$12: D3.C, D4.A
- new net N$13: D4.C, D5.A
- new net N$14: D5.C, D6.A
- new net N$15: D6.C, D7.A
- net N$4: now also J1.2
- net N$6: now also D7.C
- net N$7: now also D3.A

Commit message: save
Parts:
- removed C1: GRM32ER71J106KA12L, derek:GRM32ER71J106KA12L
- removed C2: GCM155R71H103KA55D, derek:GCM155R71H103KA55D
- removed C3: CC0805KRX7R9BB103, derek:CC0805KRX7R9BB103
- removed C4: CC0805KRX7R8BB104, derek:CC0805KRX7R8BB104
- removed C5: 08053C104KAT2A, derek:08053C104KAT2A
- removed C6: GMK212B7105KG-T, derek:GMK212B7105KG-T
- removed R1: CRCW0402121KFKED, derek:CRCW0402121KFKED
- removed R2: CRCW04027K68FKED, derek:CRCW04027K68FKED
- removed R3, R5: CRCW04021K00FKED, derek:CRCW04021K00FKED
- removed R4: CRCW0402162KFKED, derek:CRCW0402162KFKED
- removed R6: CRM0805-FX-R510ELF, derek:CRM0805-FX-R510ELF
- added CBOOT, CBOOT1: 08053C104KAT2A, derek:08053C104KAT2A
- added CCOMP, CCOMP1: CC0805KRX7R8BB104, derek:CC0805KRX7R8BB104
- added CIADJ, CIADJ1: CC0805KRX7R9BB103, derek:CC0805KRX7R9BB103
- added CIN, CIN1: GRM32ER71J106KA12L, derek:GRM32ER71J106KA12L
- added CINX, CINX1: GCM155R71H103KA55D, derek:GCM155R71H103KA55D
- added COUT, COUT1: GMK212B7105KG-T, derek:GMK212B7105KG-T
- added D10, D11, D12, D13, D14: XPGWHT, derek:XPGWHT
- added D8: PMEG6010CEH,115, derek:PMEG6010CEH,115
- added D9: BAT54WSTR, derek:BAT54WSTR
- added J2: (no value), derek:CONN_02
- added L2: 74408943220, derek:74408943220
- added RIADJ, RIADJ1, RSENSE1, RSENSE2: CRCW04021K00FKED, derek:CRCW04021K00FKED
- added RSENSE, RSENSE3: CRM0805-FX-R510ELF, derek:CRM0805-FX-R510ELF
- added RUVLOB, RUVLOB1: CRCW04027K68FKED, derek:CRCW04027K68FKED
- added RUVLOT, RUVLOT1: CRCW0402121KFKED, derek:CRCW0402121KFKED
- added R_RT, R_RT1: CRCW0402162KFKED, derek:CRCW0402162KFKED
- added U2: TPS92513HV, derek:TPS92513HV
Connections:
- removed net GND: C1.2, C2.2, C3.2, C4.2, D1.A, J1.1, R2.2, R3.2, R4.2, R6.2, U1.GND
- new net 24V: CIN.1, CIN1.1, CINX.1, CINX1.1, D2.C, D8.C, J1.2, RUVLOT.1, RUVLOT1.1, U1.VIN, U2.VIN
- new net GND-ISO: CCOMP.2, CCOMP1.2, CIADJ.2, CIADJ1.2, CIN.2, CIN1.2, CINX.2, CINX1.2, D1.A, D10.GND, D11.GND, D12.GND, D13.GND, D14.GND, D3.GND, D4.GND, D5.GND, D6.GND, D7.GND, D9.A, J1.1, RIADJ.2, RIADJ1.2, RSENSE.2, RSENSE3.2, RUVLOB.2, RUVLOB1.2, R_RT.2, R_RT1.2, U1.GND, U2.GND
- new net N$1: RUVLOB1.1, RUVLOT1.2, U2.UVLO
- new net N$16: CBOOT1.1, D9.C, L2.1, U2.PH
- new net N$17: COUT1.2, D14.C, RSENSE2.1, RSENSE3.1
- new net N$18: COUT1.1, D10.A, D8.A, L2.2
- new net N$19: R_RT1.1, U2.RT/CLK
- new net N$20: CCOMP1.1, U2.COMP
- new net N$21: CBOOT1.2, U2.BOOT
- new net N$22: RSENSE2.2, U2.ISENSE
- new net N$23: D10.C, D11.A
- new net N$24: D11.C, D12.A
- new net N$25: D12.C, D13.A
- new net N$26: D13.C, D14.A
- new net PDIM1: J2.1, U1.PDIM
- new net PDIM2: J2.2, U2.PDIM
- net N$10: now also CBOOT.2; no longer C5.2
- net N$11: now also RSENSE1.2; no longer R5.2
- net N$2: now also CIADJ.1, RIADJ.1; no longer C3.1, R3.1
- net N$3: now also RUVLOB.1, RUVLOT.2; no longer R1.2, R2.1
- net N$4: now also CIADJ1.1, RIADJ1.1, U2.IADJ; no longer C1.1, C2.1, D2.K, J1.2, R1.1, U1.VIN
- net N$5: now also CBOOT.1, D1.C; no longer C5.1, D1.K
- net N$6: now also COUT.2, RSENSE.1, RSENSE1.1; no longer C6.2, R5.1, R6.1
- net N$7: now also COUT.1; no longer C6.1
- net N$8: now also R_RT.1; no longer R4.1
- net N$9: now also CCOMP.1; no longer C4.1
Other:
- moved on the sheet: J1, L1, U1

Commit message: save
Connections:
- net N$12: now also D3.A, D7.C; no longer D3.C, D4.A
- net N$6: now also D3.C; no longer D7.C
- net N$7: now also D4.A; no longer D3.A
Other:
- moved on the sheet: D3, D4, D5, D6, D7, J1
Changed lines of the file:
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@@
 <part name="GND-ISO11" library="derek" deviceset="GND-ISO" device=""/>
 <part name="GND-ISO12" library="derek" deviceset="GND-ISO" device=""/>
+<part name="SUPPLY3" library="derek" deviceset="24V" device=""/>
+<part name="GND-ISO13" library="derek" deviceset="GND-ISO" device=""/>
 </parts>
 <sheets>
@@
 <instance part="RSENSE" gate="A" x="73.66" y="106.68" rot="R90"/>
 <instance part="COUT" gate="A" x="73.66" y="154.94" rot="R90"/>
-<instance part="D3" gate="G$1" x="91.44" y="177.8" rot="R90"/>
-<instance part="D4" gate="G$1" x="91.44" y="160.02" rot="R90"/>
-<instance part="D5" gate="G$1" x="91.44" y="142.24" rot="R90"/>
-<instance part="D6" gate="G$1" x="91.44" y="124.46" rot="R90"/>
-<instance part="D7" gate="G$1" x="91.44" y="106.68" rot="R90"/>
-<instance part="J1" gate="G$1" x="-88.9" y="121.92"/>
+<instance part="D3" gate="G$1" x="91.44" y="106.68" rot="R90"/>
+<instance part="D4" gate="G$1" x="91.44" y="177.8" rot="R90"/>
+<instance part="D5" gate="G$1" x="91.44" y="160.02" rot="R90"/>
+<instance part="D6" gate="G$1" x="91.44" y="142.24" rot="R90"/>
+<instance part="D7" gate="G$1" x="91.44" y="124.46" rot="R90"/>
+<instance part="J1" gate="G$1" x="-101.6" y="121.92"/>
 <instance part="J2" gate="G$1" x="-101.6" y="86.36"/>
 <instance part="SUPPLY1" gate="G$1" x="-73.66" y="142.24"/>
@@
 <instance part="SUPPLY2" gate="G$1" x="-73.66" y="33.02"/>
 <instance part="GND-ISO2" gate="G$1" x="-73.66" y="-10.16"/>
-<instance part="GND-ISO3" gate="G$1" x="104.14" y="167.64"/>
-<instance part="GND-ISO4" gate="G$1" x="104.14" y="149.86"/>
-<instance part="GND-ISO5" gate="G$1" x="104.14" y="129.54"/>
-<instance part="GND-ISO6" gate="G$1" x="104.14" y="111.76"/>
-<instance part="GND-ISO7" gate="G$1" x="104.14" y="93.98"/>
+<instance part="GND-ISO3" gate="G$1" x="104.14" y="96.52"/>
+<instance part="GND-ISO4" gate="G$1" x="104.14" y="167.64"/>
+<instance part="GND-ISO5" gate="G$1" x="104.14" y="147.32"/>
+<instance part="GND-ISO6" gate="G$1" x="104.14" y="129.54"/>
+<instance part="GND-ISO7" gate="G$1" x="104.14" y="111.76"/>
 <instance part="GND-ISO8" gate="G$1" x="106.68" y="-15.24"/>
 <instance part="GND-ISO9" gate="G$1" x="106.68" y="2.54"/>
@@
 <instance part="GND-ISO11" gate="G$1" x="106.68" y="38.1"/>
 <instance part="GND-ISO12" gate="G$1" x="106.68" y="63.5"/>
+<instance part="SUPPLY3" gate="G$1" x="-88.9" y="127"/>
+<instance part="GND-ISO13" gate="G$1" x="-88.9" y="116.84"/>
 </instances>
 <busses>
@@
 <wire x1="73.66" y1="142.24" x2="81.28" y2="142.24" width="0.1524" layer="91"/>
 <junction x="73.66" y="142.24"/>
-<pinref part="D7" gate="G$1" pin="C"/>
-<wire x1="91.44" y1="99.06" x2="91.44" y2="91.44" width="0.1524" layer="91"/>
 <wire x1="91.44" y1="91.44" x2="81.28" y2="91.44" width="0.1524" layer="91"/>
 <wire x1="81.28" y1="91.44" x2="81.28" y2="142.24" width="0.1524" layer="91"/>
+<pinref part="D3" gate="G$1" pin="C"/>
+<wire x1="91.44" y1="99.06" x2="91.44" y2="91.44" width="0.1524" layer="91"/>
 </segment>
 </net>
@@
 <wire x1="25.4" y1="177.8" x2="73.66" y2="177.8" width="0.1524" layer="91"/>
 <wire x1="73.66" y1="177.8" x2="73.66" y2="167.64" width="0.1524" layer="91"/>
-<pinref part="D3" gate="G$1" pin="A"/>
-<wire x1="91.44" y1="185.42" x2="91.44" y2="193.04" width="0.1524" layer="91"/>
 <wire x1="91.44" y1="193.04" x2="81.28" y2="193.04" width="0.1524" layer="91"/>
 <wire x1="81.28" y1="193.04" x2="81.28" y2="167.64" width="0.1524" layer="91"/>
 <wire x1="81.28" y1="167.64" x2="73.66" y2="167.64" width="0.1524" layer="91"/>
+<pinref part="D4" gate="G$1" pin="A"/>
+<wire x1="91.44" y1="185.42" x2="91.44" y2="193.04" width="0.1524" layer="91"/>
 </segment>
 </net>
@@
 </segment>
 </net>
-<net name="N$12" class="0">
-<segment>
-<pinref part="D3" gate="G$1" pin="C"/>
-<pinref part="D4" gate="G$1" pin="A"/>
-<wire x1="91.44" y1="170.18" x2="91.44" y2="167.64" width="0.1524" layer="91"/>
-</segment>
-</net>
 <net name="N$13" class="0">
 <segment>
 <pinref part="D4" gate="G$1" pin="C"/>
 <pinref part="D5" gate="G$1" pin="A"/>
-<wire x1="91.44" y1="152.4" x2="91.44" y2="149.86" width="0.1524" layer="91"/>
+<wire x1="91.44" y1="170.18" x2="91.44" y2="167.64" width="0.1524" layer="91"/>
 </segment>
 </net>
@@
 <pinref part="D5" gate="G$1" pin="C"/>
 <pinref part="D6" gate="G$1" pin="A"/>
-<wire x1="91.44" y1="134.62" x2="91.44" y2="132.08" width="0.1524" layer="91"/>
+<wire x1="91.44" y1="152.4" x2="91.44" y2="149.86" width="0.1524" layer="91"/>
 </segment>
 </net>
@@
 <pinref part="D6" gate="G$1" pin="C"/>
 <pinref part="D7" gate="G$1" pin="A"/>
-<wire x1="91.44" y1="116.84" x2="91.44" y2="114.3" width="0.1524" layer="91"/>
+<wire x1="91.44" y1="134.62" x2="91.44" y2="132.08" width="0.1524" layer="91"/>
 </segment>
 </net>
@@
 <junction x="40.64" y="91.44"/>
 <wire x1="-66.04" y1="106.68" x2="-73.66" y2="106.68" width="0.1524" layer="91"/>
-<wire x1="-73.66" y1="106.68" x2="-73.66" y2="121.92" width="0.1524" layer="91"/>
-<wire x1="-73.66" y1="121.92" x2="-81.28" y2="121.92" width="0.1524" layer="91"/>
 <junction x="-66.04" y="106.68"/>
-<pinref part="J1" gate="G$1" pin="1"/>
 <pinref part="GND-ISO1" gate="G$1" pin="GND-ISO"/>
 <wire x1="-73.66" y1="106.68" x2="-73.66" y2="101.6" width="0.1524" layer="91"/>
-<junction x="-73.66" y="106.68"/>
 </segment>
 <segment>
@@
 <pinref part="D7" gate="G$1" pin="GND"/>
 <pinref part="GND-ISO7" gate="G$1" pin="GND-ISO"/>
-<wire x1="96.52" y1="99.06" x2="104.14" y2="99.06" width="0.1524" layer="91"/>
-<wire x1="104.14" y1="99.06" x2="104.14" y2="96.52" width="0.1524" layer="91"/>
+<wire x1="96.52" y1="116.84" x2="104.14" y2="116.84" width="0.1524" layer="91"/>
+<wire x1="104.14" y1="116.84" x2="104.14" y2="114.3" width="0.1524" layer="91"/>
 </segment>
 <segment>
 <pinref part="D6" gate="G$1" pin="GND"/>
 <pinref part="GND-ISO6" gate="G$1" pin="GND-ISO"/>
-<wire x1="96.52" y1="116.84" x2="104.14" y2="116.84" width="0.1524" layer="91"/>
-<wire x1="104.14" y1="116.84" x2="104.14" y2="114.3" width="0.1524" layer="91"/>
+<wire x1="96.52" y1="134.62" x2="104.14" y2="134.62" width="0.1524" layer="91"/>
+<wire x1="104.14" y1="134.62" x2="104.14" y2="132.08" width="0.1524" layer="91"/>
 </segment>
 <segment>
 <pinref part="D5" gate="G$1" pin="GND"/>
 <pinref part="GND-ISO5" gate="G$1" pin="GND-ISO"/>
-<wire x1="96.52" y1="134.62" x2="104.14" y2="134.62" width="0.1524" layer="91"/>
-<wire x1="104.14" y1="134.62" x2="104.14" y2="132.08" width="0.1524" layer="91"/>
+<wire x1="96.52" y1="152.4" x2="104.14" y2="152.4" width="0.1524" layer="91"/>
+<wire x1="104.14" y1="152.4" x2="104.14" y2="149.86" width="0.1524" layer="91"/>
 </segment>
 <segment>
 <pinref part="D4" gate="G$1" pin="GND"/>
 <pinref part="GND-ISO4" gate="G$1" pin="GND-ISO"/>
-<wire x1="96.52" y1="152.4" x2="104.14" y2="152.4" width="0.1524" layer="91"/>
+<wire x1="96.52" y1="170.18" x2="104.14" y2="170.18" width="0.1524" layer="91"/>
 </segment>
 <segment>
 <pinref part="D3" gate="G$1" pin="GND"/>
 <pinref part="GND-ISO3" gate="G$1" pin="GND-ISO"/>
-<wire x1="96.52" y1="170.18" x2="104.14" y2="170.18" width="0.1524" layer="91"/>
+<wire x1="96.52" y1="99.06" x2="104.14" y2="99.06" width="0.1524" layer="91"/>
 </segment>
 <segment>
@@
 <wire x1="12.7" y1="43.18" x2="33.02" y2="43.18" width="0.1524" layer="91"/>
 </segment>
+<segment>
+<pinref part="J1" gate="G$1" pin="1"/>
+<pinref part="GND-ISO13" gate="G$1" pin="GND-ISO"/>
+<wire x1="-93.98" y1="121.92" x2="-88.9" y2="121.92" width="0.1524" layer="91"/>
+<wire x1="-88.9" y1="121.92" x2="-88.9" y2="119.38" width="0.1524" layer="91"/>
+</segment>
 </net>
 <net name="24V" class="0">
@@
 <wire x1="-66.04" y1="137.16" x2="-73.66" y2="137.16" width="0.1524" layer="91"/>
 <junction x="-66.04" y="137.16"/>
-<pinref part="J1" gate="G$1" pin="2"/>
-<wire x1="-81.28" y1="124.46" x2="-73.66" y2="124.46" width="0.1524" layer="91"/>
-<wire x1="-73.66" y1="124.46" x2="-73.66" y2="137.16" width="0.1524" layer="91"/>
 <pinref part="SUPPLY1" gate="G$1" pin="24V"/>
 <wire x1="-73.66" y1="137.16" x2="-73.66" y2="142.24" width="0.1524" layer="91"/>
-<junction x="-73.66" y="137.16"/>
 </segment>
 <segment>
@@
 <wire x1="-73.66" y1="27.94" x2="-73.66" y2="33.02" width="0.1524" layer="91"/>
 </segment>
+<segment>
+<pinref part="J1" gate="G$1" pin="2"/>
+<pinref part="SUPPLY3" gate="G$1" pin="24V"/>
+<wire x1="-93.98" y1="124.46" x2="-88.9" y2="124.46" width="0.1524" layer="91"/>
+<wire x1="-88.9" y1="124.46" x2="-88.9" y2="127" width="0.1524" layer="91"/>
+</segment>
 </net>
 <net name="PDIM1" class="0">
@@
 </segment>
 </net>
+<net name="N$12" class="0">
+<segment>
+<pinref part="D7" gate="G$1" pin="C"/>
+<pinref part="D3" gate="G$1" pin="A"/>
+<wire x1="91.44" y1="116.84" x2="91.44" y2="114.3" width="0.1524" layer="91"/>
+</segment>
+</net>

Commit message: ordered
Parts:
- renumbered D9 to GND-ISO
Changed lines of the file:
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@@
 <part name="D8" library="derek" deviceset="PMEG6010CEH,115" device=""/>
 <part name="CBOOT1" library="derek" deviceset="08053C104KAT2A" device=""/>
-<part name="D9" library="derek" deviceset="BAT54WSTR" device=""/>
+<part name="GND-ISO" library="derek" deviceset="BAT54WSTR" device=""/>
 <part name="L2" library="derek" deviceset="74408943220" device=""/>
 <part name="RSENSE2" library="derek" deviceset="CRCW04021K00FKED" device=""/>
@@
 <instance part="D8" gate="A" x="17.78" y="68.58"/>
 <instance part="CBOOT1" gate="A" x="17.78" y="58.42"/>
-<instance part="D9" gate="A" x="40.64" y="-2.54" rot="R270"/>
+<instance part="GND-ISO" gate="A" x="40.64" y="-2.54" rot="R270"/>
 <instance part="L2" gate="A" x="55.88" y="58.42"/>
 <instance part="RSENSE2" gate="A" x="55.88" y="33.02"/>
@@
 <wire x1="10.16" y1="-10.16" x2="10.16" y2="-17.78" width="0.1524" layer="91"/>
 <junction x="10.16" y="-17.78"/>
-<pinref part="D9" gate="A" pin="A"/>
+<pinref part="GND-ISO" gate="A" pin="A"/>
 <wire x1="40.64" y1="-10.16" x2="40.64" y2="-17.78" width="0.1524" layer="91"/>
 <junction x="40.64" y="-17.78"/>
@@
 <segment>
 <pinref part="L2" gate="A" pin="1"/>
-<pinref part="D9" gate="A" pin="C"/>
+<pinref part="GND-ISO" gate="A" pin="C"/>
 <wire x1="48.26" y1="58.42" x2="40.64" y2="58.42" width="0.1524" layer="91"/>
 <wire x1="40.64" y1="58.42" x2="40.64" y2="48.26" width="0.1524" layer="91"/>

Commit message: should be good to order parts
Parts:
- CBOOT, CBOOT1: value 08053C104KAT2A -> 0.1µF
- CCOMP, CCOMP1: value CC0805KRX7R8BB104 -> 0.1µF
- CIADJ, CIADJ1: value CC0805KRX7R9BB103 -> 10000pF
- CIN, CIN1: value GRM32ER71J106KA12L -> 10µF; device derek:GRM32ER71J106KA12L -> derek:GRM32ER71J106MA12L
- CINX, CINX1: value GCM155R71H103KA55D -> 10000pF
- COUT, COUT1: value GMK212B7105KG-T -> 1µF
- D1, GND-ISO: value BAT54WSTR -> BAT54WS-TP; device derek:BAT54WSTR -> derek:BAT54WS-TP
- D10, D11, D12, D13, D14: value XPGWHT -> XPGWHT-L1-0000-00G51; device derek:XPGWHT -> derek:XPGWHT-L1-0000-00G51
- D3, D4, D5, D6, D7: value XPGWHT -> XPGWHT-L1-0000-00BE8; device derek:XPGWHT -> derek:XPGWHT-L1-0000-00BE8
- L1, L2: value 74408943220 -> 22µH
- RIADJ, RIADJ1, RSENSE1, RSENSE2: value CRCW04021K00FKED -> 1k; device derek:CRCW04021K00FKED -> derek:CRCW04021K00DHEDP
- RSENSE, RSENSE3: value CRM0805-FX-R510ELF -> 0.51
- RUVLOB, RUVLOB1: value CRCW04027K68FKED -> 7.68k
- RUVLOT, RUVLOT1: value CRCW0402121KFKED -> 121k
- R_RT, R_RT1: value CRCW0402162KFKED -> 162k

Commit message: order this
Parts:
- removed GND-ISO: BAT54WS-TP, derek:BAT54WS-TP
- added CIN2, CIN3: 1µF, derek:GRM31MR71H105KA88L
- added D9: PMEG6010CEH,115, derek:PMEG6010CEH,115
- CIN, CIN1: value 10µF -> 1µF; device derek:GRM32ER71J106MA12L -> derek:GRM31MR71H105KA88L
- D1: value BAT54WS-TP -> PMEG6010CEH,115; device derek:BAT54WS-TP -> derek:PMEG6010CEH,115
- L1, L2: value 22µH -> 33µH; device derek:74408943220 -> derek:SRN6045-330M
- RIADJ, RIADJ1, RSENSE1: value 1k -> 976; device derek:CRCW04021K00DHEDP -> derek:CRCW0402976RFKED
- RSENSE2: value 1k -> 0.51; device derek:CRCW04021K00DHEDP -> derek:CRM0805-FX-R510ELF
- RSENSE3: value 0.51 -> 976; device derek:CRM0805-FX-R510ELF -> derek:CRCW0402976RFKED
- RUVLOB, RUVLOB1: value 7.68k -> 5.49k; device derek:CRCW04027K68FKED -> derek:CRCW04025K49FKED
- RUVLOT, RUVLOT1: value 121k -> 97.6k; device derek:CRCW0402121KFKED -> derek:CRCW040297K6FKED
- U1, U2: value TPS92513HV -> TPS92513; device derek:TPS92513HV -> derek:TPS92513
- renumbered R_RT to RT, R_RT1 to RT1
Connections:
- net 24V: now also CIN2.1, CIN3.1
- net GND-ISO: now also CIN2.2, CIN3.2, D9.A, RSENSE2.2; no longer GND-ISO.A, RSENSE3.2
- net N$16: now also D9.C; no longer GND-ISO.C
- net N$22: now also RSENSE3.2; no longer RSENSE2.2
