File: pwr.brd (EAGLE design)
At the start: 100 x 80 mm, 43 parts, among them Q1 IPD65R600E6, T1 750811647, U1 UCC28700

Commit message: wip
Parts:
- moved U$9 10.4 mm to (85.0, 34.0)
- moved U$3 6.73 mm to (47.5, 22.0)
- moved F1 6.10 mm to (41.5, 27.0)
- moved R10 5.83 mm to (37.0, 44.0)
- moved R9 5.83 mm to (40.0, 44.0)
- moved U$2 5.59 mm to (37.5, 22.0)
- moved D3 5.41 mm to (46.0, 32.0)
- moved R7 5.02 mm to (50.5, 43.0), turned to 270 degrees
- moved C7 4.30 mm to (41.5, 39.5), turned to 0 degrees
- moved Q1 4.03 mm to (46.0, 48.5)
- moved C9 3.54 mm to (55.5, 34.0)
- moved C1 3.20 mm to (67.0, 28.0)
- moved C6 3.04 mm to (85.0, 30.5), turned to 270 degrees
- moved R1 3.00 mm to (79.5, 28.5)
- moved R101 3.00 mm to (79.5, 26.0)
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Routing:
- net GND: track 0.00 -> 26.1 mm
- net N$15: track 0.00 -> 22.7 mm
- net N$17: track 0.00 -> 19.6 mm, vias 0 -> 1
- net N$10: track 0.00 -> 19.4 mm
- net N$14: track 0.00 -> 16.2 mm, vias 0 -> 2
- net N$3: track 0.00 -> 14.8 mm
- net N$13: track 0.00 -> 10.7 mm
- net N$2: track 0.00 -> 7.75 mm
- net N$11: track 0.00 -> 7.73 mm
- net N$1: track 0.00 -> 4.48 mm
- net N$6: track 0.00 -> 4.36 mm
- net N$20: track 0.00 -> 4.35 mm
- net N$9: track 0.00 -> 3.40 mm
- net N$18: track 0.00 -> 3.19 mm
- net N$8: track 0.00 -> 3.00 mm
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- added copper zone on layer 16, net 24V
- added copper zone on layer 16, net GND
- added copper zone on layer 16, net GND-ISO

Commit message: save
Parts:
- removed U$5, U$6, U$7: TP-1502, derek:TP-1502
- moved U$8 86.0 mm to (81.7, 45.4)
- moved C_2 76.7 mm to (77.4, 39.6), flipped to the bottom
- moved L_1 74.7 mm to (77.1, 43.2), flipped to the bottom
- moved C_1 71.5 mm to (74.8, 36.9), flipped to the bottom
- moved U_1 69.7 mm to (74.1, 39.4), flipped to the bottom
- moved R_1 68.2 mm to (73.6, 41.5), flipped to the bottom
- moved C8 18.0 mm to (40.5, 39.5)
- moved C9 18.0 mm to (38.0, 38.0)
- moved D1 18.0 mm to (62.0, 40.5)
- moved D2 18.0 mm to (38.0, 57.0)
- moved D3 18.0 mm to (28.5, 36.0)
- moved D4 18.0 mm to (43.0, 55.0)
- moved D5 18.0 mm to (36.0, 36.0)
- moved F1 18.0 mm to (24.0, 31.0)
- moved Q1 18.0 mm to (28.5, 52.5)
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Connections:
- net 24V: no longer U$5.1
- net GND-ISO: no longer U$6.1, U$7.1
Routing:
- net N$3: track 14.8 -> 57.4 mm
- net GND: track 26.1 -> 0.60 mm
- net N$10: track 19.4 -> 0.80 mm
- net 3.3V: track 0.00 -> 18.1 mm, vias 0 -> 2
- net 24V: track 0.00 -> 8.61 mm
- net GND-ISO: track 0.00 -> 4.35 mm
- net N$5: track 0.00 -> 3.83 mm
- net N$16: track 0.00 -> 1.94 mm
- net N$4: track 0.00 -> 1.91 mm
- net N$17: track 19.6 -> 21.2 mm, vias 1 -> 2
- added copper zone on layer 16, net N$10

Commit message: update lib
Other:
- board size 100 x 80 mm -> 50 x 58 mm
Changed lines of the file:
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@@
 <board>
 <plain>
-<wire x1="0" y1="0" x2="100" y2="0" width="0" layer="20"/>
-<wire x1="100" y1="0" x2="100" y2="80" width="0" layer="20"/>
-<wire x1="100" y1="80" x2="0" y2="80" width="0" layer="20"/>
-<wire x1="0" y1="80" x2="0" y2="0" width="0" layer="20"/>
-<wire x1="19.791" y1="58.122" x2="19.791" y2="32.522" width="0.001" layer="121"/>
-<wire x1="35.083859375" y1="59.322" x2="50.080859375" y2="65.622" width="0.001" layer="121" curve="45.572997"/>
-<wire x1="35.083859375" y1="59.322" x2="23.791" y2="59.322" width="0.001" layer="121"/>
-<wire x1="23.791" y1="59.322" x2="21.95796875" y2="58.122" width="0.001" layer="121" curve="66.421833"/>
-<wire x1="19.791" y1="58.122" x2="21.95796875" y2="58.122" width="0.001" layer="121"/>
-<wire x1="69.791" y1="74.30475" x2="69.791" y2="16.33925" width="0.001" layer="121"/>
-<wire x1="69.791" y1="74.30475" x2="50.0808625" y2="65.622" width="0.001" layer="121" curve="43.596881"/>
-<wire x1="50.080859375" y1="25.022" x2="35.083859375" y2="31.322" width="0.001" layer="121" curve="45.572997"/>
-<wire x1="50.080859375" y1="25.022" x2="69.791" y2="16.339246875" width="0.001" layer="121" curve="43.596885"/>
-<wire x1="35.083859375" y1="31.322" x2="23.791" y2="31.322" width="0.001" layer="121"/>
-<wire x1="19.791" y1="32.522" x2="21.95796875" y2="32.522" width="0.001" layer="121"/>
-<wire x1="21.95796875" y1="32.522" x2="23.791" y2="31.322" width="0.001" layer="121" curve="66.421833"/>
+<wire x1="19.791" y1="58.122" x2="19.791" y2="32.522" width="0.001" layer="20"/>
+<wire x1="35.083859375" y1="59.322" x2="50.080859375" y2="65.622" width="0.001" layer="20" curve="45.572997"/>
+<wire x1="35.083859375" y1="59.322" x2="23.791" y2="59.322" width="0.001" layer="20"/>
+<wire x1="23.791" y1="59.322" x2="21.95796875" y2="58.122" width="0.001" layer="20" curve="66.421833"/>
+<wire x1="19.791" y1="58.122" x2="21.95796875" y2="58.122" width="0.001" layer="20"/>
+<wire x1="69.791" y1="74.30475" x2="69.791" y2="16.33925" width="0.001" layer="20"/>
+<wire x1="69.791" y1="74.30475" x2="50.0808625" y2="65.622" width="0.001" layer="20" curve="43.596881"/>
+<wire x1="50.080859375" y1="25.022" x2="35.083859375" y2="31.322" width="0.001" layer="20" curve="45.572997"/>
+<wire x1="50.080859375" y1="25.022" x2="69.791" y2="16.339246875" width="0.001" layer="20" curve="43.596885"/>
+<wire x1="35.083859375" y1="31.322" x2="23.791" y2="31.322" width="0.001" layer="20"/>
+<wire x1="19.791" y1="32.522" x2="21.95796875" y2="32.522" width="0.001" layer="20"/>
+<wire x1="21.95796875" y1="32.522" x2="23.791" y2="31.322" width="0.001" layer="20" curve="66.421833"/>
 </plain>
 <attributes>
@@
 <vertex x="33" y="27"/>
 </polygon>
+<wire x1="22.5" y1="46.6" x2="19.5" y2="46.6" width="0" layer="19" extent="16-16"/>
 </signal>
 <signal name="N$2">
@@
 <wire x1="40" y1="49.5" x2="40" y2="49.6" width="0.4064" layer="16"/>
 <wire x1="45" y1="49.6" x2="45" y2="48.9017" width="0.4064" layer="16"/>
-<polygon width="0.4064" layer="16">
+<polygon width="0.4064" layer="16" thermals="no">
 <vertex x="33.5" y="59.5"/>
 <vertex x="17.5" y="59.5"/>
@@
 <wire x1="73.57" y1="38.44" x2="73.57" y2="39.39" width="0.4064" layer="16"/>
 <wire x1="73.57" y1="39.39" x2="74.07" y2="39.39" width="0.4064" layer="16"/>
+<wire x1="68.5" y1="33.0983" x2="71" y2="31.5" width="0" layer="19" extent="16-16"/>
+<wire x1="75.5385" y1="36.85" x2="71" y2="31.5" width="0" layer="19" extent="16-16"/>
 </signal>
 <signal name="24V">

Commit message: getting close
Parts:
- added U2: ESP3212, derek:QFN48-0.4MM
- C1: value DE1E3KX222MA4BL01 -> 2200pF
- C2, C3: value UHE1V221MPD6 -> 220µF
- C4, C5: value UMK316AB7475KL-T -> 4.7µF
- C6: value 08053C104KAT2A -> 0.1µF
- C7: value EEUED2G470 -> 47µF
- C8: value 06035C104KAT2A -> 0.1µF
- C9: value GRM31CR61H225KA88L -> 2.2µF
- C_1: value C1608X5R1V225K080AC -> 2.2µF
- C_2: value GRM21BR60J226ME39L -> 22µF
- Q1: value IPD65R600E6 -> IPD65R600C6
- R1, R101: value CRCW120610K0JNEA -> 10k
- R10, R9: value CSR1206FKR750 -> 0.75
- R11: value CRCW060319K6FKEA -> 19.6k
- R2: value CRCW120633R2FKEA -> 33.2; device derek:1206 -> derek:1210
- R3: value CRCW12064R70JNEA -> 4.7
- R4: value CRCW060375K0FKEA -> 75k
- R5, R6: value CRCW08053M30JNEA -> 3.3M
- R7: value CRCW06030000Z0EA -> 0.0
- R8: value CRCW1206698RFKEA -> 698
- R_1: value CRCW0402100KFKED -> 100k
- moved U$3 24.4 mm to (9.00, 38.5)
- moved F1 23.6 mm to (10.0, 50.0), flipped to the bottom, turned to 180 degrees
- moved U$2 19.0 mm to (9.00, 41.5)
- moved D3 11.0 mm to (18.5, 40.5), turned to 270 degrees
- moved U$8 8.94 mm to (73.7, 49.4)
- moved R10 8.14 mm to (25.0, 42.0)
- moved R9 7.81 mm to (27.5, 42.0)
- moved C_1 4.50 mm to (70.3, 36.9)
- moved C_2 4.50 mm to (72.9, 39.6)
- moved L_1 4.50 mm to (72.6, 43.2)
- moved R_1 4.50 mm to (69.1, 41.5)
- moved U_1 4.50 mm to (69.6, 39.4)
- moved U$10 4.47 mm to (67.0, 29.5)
- moved C7 3.61 mm to (21.5, 41.5), turned to 300 degrees
- moved R4 3.50 mm to (41.5, 38.0)
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Connections:
- net N$14: now also D5.C; no longer D5.1
- net N$16: now also D5.A; no longer D5.2
Routing:
- net N$3: track 57.4 -> 32.5 mm
- net N$1: track 4.48 -> 10.3 mm
- net 3.3V: track 18.1 -> 20.4 mm
- net N$15: track 22.7 -> 24.8 mm
- net N$13: track 10.7 -> 9.11 mm
- net 24V: track 8.61 -> 7.08 mm
- net N$17: track 21.2 -> 20.3 mm
- net N$11: track 7.73 -> 8.62 mm
- net GND: track 0.60 -> 0.00 mm
- net N$10: track 0.80 -> 0.26 mm
Other:
- board size 50 x 58 mm -> 70.3 x 58 mm

Commit message: pwr to osh
Parts:
- removed U2: ESP3212, derek:QFN48-0.4MM
- L_1: value LPS4018-103MRBLPS4018-103MRB -> 10µH; device derek:LPS4018 -> derek:SDR0503
- moved R7 5.39 mm to (26.0, 45.0)
- moved Q1 2.24 mm to (24.5, 49.5), turned to 90 degrees
- moved C7 1.80 mm to (20.0, 42.5), turned to 315 degrees
- moved L_1 1.02 mm to (72.8, 44.2)
- moved R10 1.00 mm to (25.0, 41.0)
- moved R9 1.00 mm to (27.5, 41.0)
Routing:
- net N$13: track 9.11 -> 15.3 mm
- net N$12: track 2.49 -> 5.89 mm
- net N$15: track 24.8 -> 27.5 mm
- net N$3: track 32.5 -> 30.9 mm
- net N$1: track 10.3 -> 9.47 mm
- net 3.3V: track 20.4 -> 21.2 mm
Other:
- outline, holes or cut-outs redrawn

Commit message: save
Parts:
- added U$1, U$4, U$5: TP-1502, derek:TP-1502
- added U3: ESP-WROOM-32, derek:ESP-WROOM-32
- moved U$10 38.6 mm to (74.0, 67.5)
- moved U$9 30.2 mm to (74.0, 70.0)
- moved C3 11.1 mm to (57.0, 56.5)
- moved U$8 8.12 mm to (74.0, 57.5)
- moved C2 4.30 mm to (57.0, 33.5)
- moved C1 3.81 mm to (43.5, 32.0)
- moved C4 3.81 mm to (56.5, 47.5)
- moved C5 3.81 mm to (56.5, 50.5)
- moved C6 3.81 mm to (62.0, 32.5)
- moved C8 3.81 mm to (34.0, 38.0)
- moved C9 3.81 mm to (31.5, 36.5)
- moved C_1 3.81 mm to (66.8, 35.4)
- moved C_2 3.81 mm to (69.4, 38.1)
- moved D1 3.81 mm to (55.5, 39.0)
- moved D2 3.81 mm to (31.5, 55.5)
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Connections:
- new net N$21: U$1.1, U3.10
- new net N$23: U$5.1, U3.12
- new net N$24: U$4.1, U3.11
- net 3.3V: now also U3.2
- net GND: now also U1.5
- net GND-ISO: now also U3.1, U3.15, U3.38, U3.GND
Routing:
- net 24V: track 7.08 -> 27.5 mm
- net N$23: track 0.00 -> 18.7 mm
- net N$24: track 0.00 -> 16.1 mm
- net N$21: track 0.00 -> 13.7 mm
- net 3.3V: track 21.2 -> 30.9 mm, vias 2 -> 3
- net GND-ISO: track 4.35 -> 0.00 mm, vias 0 -> 7
- net N$3: track 30.9 -> 26.9 mm
- net N$2: track 7.32 -> 3.95 mm
- net N$15: track 27.5 -> 26.2 mm
- net N$1: track 9.47 -> 10.2 mm
- added copper zone on layer 1, net GND-ISO
Other:
- board size 70.3 x 58 mm -> 78.5 x 58 mm

Commit message: save
Parts:
- moved D3 14.5 mm to (21.5, 52.0)
- moved U$2 12.2 mm to (7.00, 53.5)
- moved R7 12.0 mm to (34.0, 47.0)
- moved U$3 11.2 mm to (7.00, 49.5)
- moved C7 9.12 mm to (29.0, 41.0), turned to 270 degrees
- moved Q1 8.94 mm to (29.0, 52.0), turned to 0 degrees
- moved C1 4.74 mm to (48.0, 33.5)
- moved C2 4.74 mm to (61.5, 35.0)
- moved C3 4.74 mm to (61.5, 58.0)
- moved C4 4.74 mm to (61.0, 49.0)
- moved C5 4.74 mm to (61.0, 52.0)
- moved C6 4.74 mm to (66.5, 34.0)
- moved C8 4.74 mm to (38.5, 39.5)
- moved C9 4.74 mm to (36.0, 38.0)
- moved C_1 4.74 mm to (71.3, 36.9)
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Routing:
- net N$3: track 26.9 -> 2.82 mm
- net N$15: track 26.2 -> 12.8 mm
- net N$13: track 15.3 -> 3.75 mm
- net N$2: track 3.95 -> 13.9 mm
- net N$12: track 5.89 -> 0.00 mm
- net 3.3V: track 30.9 -> 35.9 mm
- net 24V: track 27.5 -> 31.5 mm
- net N$1: track 10.2 -> 6.32 mm
- net N$23: track 18.7 -> 21.4 mm
- net N$11: track 8.62 -> 6.24 mm
- net N$24: track 16.1 -> 16.7 mm
Other:
- board size 78.5 x 58 mm -> 79.5 x 58 mm

Commit message: save
Changed lines of the file:
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@@
 <element name="U_1" library="derek" package="P-WSON(10)" value="TPS62177" x="70.57" y="39.39" rot="MR0">
 <attribute name="DATASHEET_URL" value="http://www.ti.com/lit/ds/symlink/tps62177.pdf" x="70.57" y="39.39" size="1.778" layer="28" rot="MR0" display="off"/>
-<attribute name="DIGIKEY_PART_NUMBER" value="296-41856-6-ND" x="70.57" y="39.39" size="1.778" layer="28" rot="MR0" display="off"/>
+<attribute name="DIGIKEY_PART_NUMBER" value="296-41856-1-ND" x="70.57" y="39.39" size="1.778" layer="28" rot="MR0" display="off"/>
 <attribute name="MANUFACTURER" value="Texas Instruments" x="70.57" y="39.39" size="1.778" layer="28" rot="MR0" display="off"/>
 <attribute name="PART_NUMBER" value="TPS62177DQCR" x="70.57" y="39.39" size="1.778" layer="28" rot="MR0" display="off"/>
@@
 <element name="C1" library="derek" package="DE1E3KX222MA4BL01" value="2200pF" x="48" y="33.5" rot="R180">
 <attribute name="DATASHEET_URL" value="http://www.murata.com/~/media/webrenewal/support/library/catalog/products/capacitor/mlcc/c85e.ashx" x="48" y="33.5" size="1.778" layer="27" rot="R180" display="off"/>
-<attribute name="DIGIKEY_PART_NUMBER" value="490-7047-ND" x="48" y="33.5" size="1.778" layer="27" rot="R180" display="off"/>
+<attribute name="DIGIKEY_PART_NUMBER" value="490-9384-ND" x="48" y="33.5" size="1.778" layer="27" rot="R180" display="off"/>
 <attribute name="MANUFACTURER" value="Murata Electronics North America" x="48" y="33.5" size="1.778" layer="27" rot="R180" display="off"/>
 <attribute name="PART_NUMBER" value="DE1E3KX222MA4BN01F" x="48" y="33.5" size="1.778" layer="27" rot="R180" display="off"/>
@@
 <attribute name="DATASHEET_URL" value="http://datasheets.avx.com/X7RDielectric.pdf" x="66.5" y="34" size="1.778" layer="28" rot="MR270" display="off"/>
 <attribute name="DIGIKEY_PART_NUMBER" value="478-3755-1-ND" x="66.5" y="34" size="1.778" layer="28" rot="MR270" display="off"/>
+<attribute name="MANUFACTURER" value="AVX Corporation" x="66.5" y="34" size="1.778" layer="28" rot="MR270" display="off"/>
 <attribute name="PART_NUMBER" value="08053C104KAT2A" x="66.5" y="34" size="1.778" layer="28" rot="MR270" display="off"/>
 <attribute name="VALUE" value="0.1µF" x="66.5" y="34" size="1.778" layer="28" rot="MR270" display="off"/>
@@
 <contactref element="F1" pad="2"/>
 <wire x1="19.1" y1="53.35" x2="15.1" y2="50.27" width="0.4064" layer="16"/>
-<wire x1="15.1" y1="50.27" x2="14.77" y2="51.5" width="0.4064" layer="16"/>
+<wire x1="15.1" y1="50.27" x2="16.04" y2="51.5" width="0.4064" layer="16"/>
 </signal>
 <signal name="N$3">
@@
 <contactref element="U$2" pad="1"/>
 <contactref element="F1" pad="1"/>
-<wire x1="12.23" y1="51.5" x2="11.23" y2="53.23" width="0.4064" layer="16"/>
+<wire x1="10.96" y1="51.5" x2="11.23" y2="53.23" width="0.4064" layer="16"/>
 <wire x1="11.23" y1="53.23" x2="7" y2="53.5" width="0.4064" layer="16"/>
 </signal>
