File: pwr.brd (EAGLE design)
At the start: 79.5 x 58 mm, 44 parts, among them Q1 IPD65R600C6, T1 750811647, U1 UCC28700, U3 ESP-WROOM-32

Commit message: save
Parts:
- moved R10 1.50 mm to (27.5, 41.0)
- moved R9 1.00 mm to (29.5, 41.0)
- turned D1 to 0 degrees
Connections:
- net N$3: now also D2.A; no longer D2.2
- net N$8: now also D2.C, D4.C; no longer D2.1, D4.1
- net N$9: now also D4.A; no longer D4.2
Routing:
- net GND: track 0.00 -> 13.1 mm
- net 3.3V: track 35.9 -> 29.2 mm
- net N$15: track 12.8 -> 17.3 mm
- net N$13: track 3.75 -> 7.48 mm
- net N$12: track 0.00 -> 2.31 mm
- net N$14: track 16.3 -> 15.6 mm

Commit message: sent
Parts:
- moved R10 0.50 mm to (27.0, 41.0)
- flipped F1 to the top
Routing:
- net N$11: track 5.99 -> 9.35 mm, vias 0 -> 1
- net N$1: track 6.60 -> 8.94 mm, vias 0 -> 1
Changed lines of the file:
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@@
 <attribute name="VALUE" value="0.75" x="29.5" y="41" size="1.778" layer="28" rot="MR270" display="off"/>
 </element>
-<element name="R10" library="derek" package="1206" value="0.75" x="27.5" y="41" rot="MR270">
-<attribute name="DATASHEET_URL" value="https://www.seielect.com/Catalog/SEI-CSR_CSRN.pdf" x="27.5" y="41" size="1.778" layer="28" rot="MR270" display="off"/>
-<attribute name="DIGIKEY_PART_NUMBER" value="CSR1206FKR750CT-ND" x="27.5" y="41" size="1.778" layer="28" rot="MR270" display="off"/>
-<attribute name="MANUFACTURER" value="Stackpole Electronics Inc." x="27.5" y="41" size="1.778" layer="28" rot="MR270" display="off"/>
-<attribute name="PART_NUMBER" value="CSR1206FKR750" x="27.5" y="41" size="1.778" layer="28" rot="MR270" display="off"/>
-<attribute name="VALUE" value="0.75" x="27.5" y="41" size="1.778" layer="28" rot="MR270" display="off"/>
+<element name="R10" library="derek" package="1206" value="0.75" x="27" y="41" rot="MR270">
+<attribute name="DATASHEET_URL" value="https://www.seielect.com/Catalog/SEI-CSR_CSRN.pdf" x="27" y="41" size="1.778" layer="28" rot="MR270" display="off"/>
+<attribute name="DIGIKEY_PART_NUMBER" value="CSR1206FKR750CT-ND" x="27" y="41" size="1.778" layer="28" rot="MR270" display="off"/>
+<attribute name="MANUFACTURER" value="Stackpole Electronics Inc." x="27" y="41" size="1.778" layer="28" rot="MR270" display="off"/>
+<attribute name="PART_NUMBER" value="CSR1206FKR750" x="27" y="41" size="1.778" layer="28" rot="MR270" display="off"/>
+<attribute name="VALUE" value="0.75" x="27" y="41" size="1.778" layer="28" rot="MR270" display="off"/>
 </element>
 <element name="C1" library="derek" package="DE1E3KX222MA4BL01" value="2200pF" x="48" y="33.5" rot="R180">
@@
 <attribute name="VALUE" value="10k" x="61" y="30" size="1.778" layer="28" rot="MR0" display="off"/>
 </element>
-<element name="F1" library="derek" package="TR5_FUSE_8.5" value="37012000410" x="13.5" y="51.5" rot="MR180">
-<attribute name="DATASHEET_URL" value="http://www.littelfuse.com/~/media/electronics/datasheets/fuses/littelfuse_fuse_370_datasheet.pdf.pdf" x="13.5" y="51.5" size="1.778" layer="28" rot="MR180" display="off"/>
-<attribute name="DIGIKEY_PART_NUMBER" value="WK4957BK-ND" x="13.5" y="51.5" size="1.778" layer="28" rot="MR180" display="off"/>
-<attribute name="MANUFACTURER" value="Littelfuse Inc." x="13.5" y="51.5" size="1.778" layer="28" rot="MR180" display="off"/>
-<attribute name="PART_NUMBER" value="37012000410" x="13.5" y="51.5" size="1.778" layer="28" rot="MR180" display="off"/>
+<element name="F1" library="derek" package="TR5_FUSE_8.5" value="37012000410" x="13.5" y="51.5" rot="R180">
+<attribute name="DATASHEET_URL" value="http://www.littelfuse.com/~/media/electronics/datasheets/fuses/littelfuse_fuse_370_datasheet.pdf.pdf" x="13.5" y="51.5" size="1.778" layer="27" rot="R180" display="off"/>
+<attribute name="DIGIKEY_PART_NUMBER" value="WK4957BK-ND" x="13.5" y="51.5" size="1.778" layer="27" rot="R180" display="off"/>
+<attribute name="MANUFACTURER" value="Littelfuse Inc." x="13.5" y="51.5" size="1.778" layer="27" rot="R180" display="off"/>
+<attribute name="PART_NUMBER" value="37012000410" x="13.5" y="51.5" size="1.778" layer="27" rot="R180" display="off"/>
 </element>
 <element name="U3" library="derek" package="ESP-WROOM-32" value="ESP-WROOM-32" x="68" y="44.5"/>
@@
 </polygon>
 <contactref element="U1" pad="5"/>
-<wire x1="23.9" y1="50.65" x2="23.9" y2="41.7" width="0.4064" layer="16"/>
-<wire x1="23.9" y1="41.7" x2="27.5" y2="39.6" width="0.4064" layer="16"/>
+<wire x1="24.45" y1="50.65" x2="23.9" y2="41.7" width="0.4064" layer="16"/>
+<wire x1="23.9" y1="41.7" x2="27" y2="39.6" width="0.4064" layer="16"/>
 </signal>
 <signal name="N$2">
 <contactref element="U$3" pad="1"/>
 <contactref element="D3" pad="3"/>
-<wire x1="19.1" y1="50.65" x2="11.85" y2="46.65" width="0.4064" layer="16"/>
+<wire x1="18.55" y1="50.65" x2="11.85" y2="46.65" width="0.4064" layer="16"/>
 <wire x1="11.85" y1="46.65" x2="7" y2="49.5" width="0.4064" layer="16"/>
 </signal>
@@
 <contactref element="D3" pad="4"/>
 <contactref element="F1" pad="2"/>
-<wire x1="19.1" y1="53.35" x2="15.1" y2="50.27" width="0.4064" layer="16"/>
-<wire x1="15.1" y1="50.27" x2="16.04" y2="51.5" width="0.4064" layer="16"/>
+<wire x1="18.55" y1="53.35" x2="15.1" y2="50.27" width="0.4064" layer="16"/>
+<wire x1="15.1" y1="50.27" x2="10.96" y2="51.5" width="0.4064" layer="1"/>
+<via x="15.1" y="50.27" extent="1-16" drill="0.35"/>
 </signal>
 <signal name="N$3">
@@
 <wire x1="33.5" y1="57" x2="33.8" y2="57" width="0.4064" layer="16"/>
 <wire x1="33.5" y1="54.48" x2="33.5" y2="57" width="0.4064" layer="16"/>
-<wire x1="23.9" y1="53.35" x2="33.5" y2="54.48" width="0" layer="19" extent="16-16"/>
-<wire x1="29" y1="44.75" x2="23.9" y2="53.35" width="0" layer="19" extent="16-16"/>
+<wire x1="24.45" y1="53.35" x2="33.5" y2="54.48" width="0" layer="19" extent="16-16"/>
+<wire x1="29" y1="44.75" x2="24.45" y2="53.35" width="0" layer="19" extent="16-16"/>
 </signal>
 <signal name="N$7">
@@
 <contactref element="D4" pad="A"/>
 <contactref element="R2" pad="2"/>
-<wire x1="38" y1="52.755" x2="41" y2="52.4" width="0.4064" layer="16"/>
+<wire x1="38" y1="52.4" x2="41" y2="52.4" width="0.4064" layer="16"/>
 <wire x1="41" y1="52.4" x2="41" y2="52.8" width="0.4064" layer="16"/>
 </signal>
@@
 <contactref element="Q1" pad="2"/>
 <contactref element="R6" pad="1"/>
-<wire x1="38" y1="49.5" x2="38" y2="49.245" width="0.4064" layer="16"/>
+<wire x1="38" y1="49.5" x2="38" y2="49.6" width="0.4064" layer="16"/>
 <polygon width="0.4064" layer="16" thermals="no">
 <vertex x="30.5" y="55.5"/>
@@
 <contactref element="R9" pad="1"/>
 <contactref element="R10" pad="1"/>
-<wire x1="27.5" y1="42.4" x2="29.5" y2="42.4" width="0.4064" layer="16"/>
+<wire x1="27" y1="42.4" x2="29.5" y2="42.4" width="0.4064" layer="16"/>
 <wire x1="37.1" y1="45" x2="34.9748125" y2="45" width="0.4064" layer="16"/>
 <wire x1="34.9748125" y1="45" x2="34.0784125" y2="45.8964" width="0.4064" layer="16"/>
@@
 <wire x1="32.4964" y1="45.8964" x2="29.5" y2="42.4" width="0.4064" layer="16"/>
 <wire x1="26.7" y1="47.8" x2="26.7" y2="43.1" width="0.4064" layer="16"/>
-<wire x1="26.7" y1="43.1" x2="27.5" y2="42.4" width="0.4064" layer="16"/>
+<wire x1="26.7" y1="43.1" x2="27" y2="42.4" width="0.4064" layer="16"/>
 </signal>
 <signal name="N$16">
@@
 <contactref element="U$2" pad="1"/>
 <contactref element="F1" pad="1"/>
-<wire x1="10.96" y1="51.5" x2="11.23" y2="53.23" width="0.4064" layer="16"/>
+<wire x1="16.04" y1="51.5" x2="11.23" y2="53.23" width="0.4064" layer="1"/>
 <wire x1="11.23" y1="53.23" x2="7" y2="53.5" width="0.4064" layer="16"/>
+<via x="11.23" y="53.23" extent="1-16" drill="0.35"/>
 </signal>
 <signal name="N$23">

Commit message: save
Parts:
- flipped F1 to the bottom
Routing:
- net N$11: track 9.35 -> 5.99 mm
- net N$1: track 8.94 -> 6.17 mm
Changed lines of the file:
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@@
 <attribute name="VALUE" value="10k" x="61" y="30" size="1.778" layer="28" rot="MR0" display="off"/>
 </element>
-<element name="F1" library="derek" package="TR5_FUSE_8.5" value="37012000410" x="13.5" y="51.5" rot="R180">
-<attribute name="DATASHEET_URL" value="http://www.littelfuse.com/~/media/electronics/datasheets/fuses/littelfuse_fuse_370_datasheet.pdf.pdf" x="13.5" y="51.5" size="1.778" layer="27" rot="R180" display="off"/>
-<attribute name="DIGIKEY_PART_NUMBER" value="WK4957BK-ND" x="13.5" y="51.5" size="1.778" layer="27" rot="R180" display="off"/>
-<attribute name="MANUFACTURER" value="Littelfuse Inc." x="13.5" y="51.5" size="1.778" layer="27" rot="R180" display="off"/>
-<attribute name="PART_NUMBER" value="37012000410" x="13.5" y="51.5" size="1.778" layer="27" rot="R180" display="off"/>
+<element name="F1" library="derek" package="TR5_FUSE_8.5" value="37012000410" x="13.5" y="51.5" rot="MR180">
+<attribute name="DATASHEET_URL" value="http://www.littelfuse.com/~/media/electronics/datasheets/fuses/littelfuse_fuse_370_datasheet.pdf.pdf" x="13.5" y="51.5" size="1.778" layer="28" rot="MR180" display="off"/>
+<attribute name="DIGIKEY_PART_NUMBER" value="WK4957BK-ND" x="13.5" y="51.5" size="1.778" layer="28" rot="MR180" display="off"/>
+<attribute name="MANUFACTURER" value="Littelfuse Inc." x="13.5" y="51.5" size="1.778" layer="28" rot="MR180" display="off"/>
+<attribute name="PART_NUMBER" value="37012000410" x="13.5" y="51.5" size="1.778" layer="28" rot="MR180" display="off"/>
 </element>
 <element name="U3" library="derek" package="ESP-WROOM-32" value="ESP-WROOM-32" x="68" y="44.5"/>
@@
 <contactref element="F1" pad="2"/>
 <wire x1="18.55" y1="53.35" x2="15.1" y2="50.27" width="0.4064" layer="16"/>
-<wire x1="15.1" y1="50.27" x2="10.96" y2="51.5" width="0.4064" layer="1"/>
+<wire x1="15.1" y1="50.27" x2="16.04" y2="51.5" width="0.4064" layer="16"/>
 <via x="15.1" y="50.27" extent="1-16" drill="0.35"/>
 </signal>
@@
 <contactref element="U$2" pad="1"/>
 <contactref element="F1" pad="1"/>
-<wire x1="16.04" y1="51.5" x2="11.23" y2="53.23" width="0.4064" layer="1"/>
+<wire x1="10.96" y1="51.5" x2="11.23" y2="53.23" width="0.4064" layer="16"/>
 <wire x1="11.23" y1="53.23" x2="7" y2="53.5" width="0.4064" layer="16"/>
 <via x="11.23" y="53.23" extent="1-16" drill="0.35"/>

Commit message: ordered
Parts:
- added U$6: 10k, derek:0603
- moved U$2 51.2 mm to (3.60, 2.40)
- moved U$3 47.5 mm to (14.4, 2.60)
- moved U$9 45.6 mm to (52.7, 30.2)
- moved F1 43.9 mm to (8.10, 7.90)
- moved U$10 40.0 mm to (49.3, 36.5)
- moved D3 39.5 mm to (11.1, 13.9), turned to 180 degrees
- moved U$5 38.1 mm to (60.4, 29.9)
- moved C3 36.4 mm to (48.1, 24.2)
- moved U$4 34.9 mm to (62.9, 29.9)
- moved U$1 31.8 mm to (65.4, 29.9)
- moved C7 29.0 mm to (8.70, 20.3), turned to 0 degrees
- moved U$8 28.1 mm to (74.3, 29.9)
- moved R9 28.0 mm to (6.20, 25.4)
- moved R7 26.8 mm to (17.2, 26.1), turned to 270 degrees
- moved Q1 26.5 mm to (12.9, 31.0)
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Connections:
- new net N$22: U$6.1, U3.3
- net 3.3V: now also U$6.2
Routing:
- net 24V: track 31.5 -> 11.7 mm
- net N$23: track 21.4 -> 3.21 mm
- net N$24: track 16.7 -> 2.70 mm
- net GND: track 12.7 -> 0.00 mm
- net N$21: track 14.0 -> 3.21 mm
- net N$10: track 0.10 -> 5.11 mm, vias 0 -> 21
- net N$2: track 13.4 -> 9.16 mm
- net N$13: track 7.48 -> 11.5 mm
- net N$9: track 3.40 -> 0.00 mm, vias 0 -> 5
- net N$8: track 3.00 -> 0.00 mm, vias 0 -> 8
- net N$3: track 2.82 -> 0.00 mm, vias 0 -> 7
- net N$1: track 6.17 -> 3.42 mm, vias 1 -> 0
- net N$15: track 17.5 -> 14.8 mm
- net N$22: track 0.00 -> 2.45 mm
- net 3.3V: track 29.2 -> 31.5 mm, vias 3 -> 2
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- added copper zone on layer 1, net N$10
- added copper zone on layer 16, net N$15
- added copper zone on layer 1, net N$3
- added copper zone on layer 16, net N$3
- added copper zone on layer 1, net N$8
- added copper zone on layer 16, net N$8
- added copper zone on layer 1, net N$9
- added copper zone on layer 16, net N$9
Other:
- board size 79.5 x 58 mm -> 77.2 x 41 mm

Commit message: works
Parts:
- moved L_1 0.13 mm to (64.4, 33.9)
- moved C_1 0.06 mm to (56.6, 36.6)
Connections:
- net GND-ISO: now also U_1.P$1, U_1.P$10, U_1.P$2
Other:
- board size 77.2 x 41 mm -> 132.6 x 103.3 mm

Commit message: temp
Parts:
- removed R7: 0.0, derek:0603
- moved U$10 39.6 mm to (84.5, 18.3)
- moved C7 24.2 mm to (32.9, 20.0)
- moved U3 24.1 mm to (81.7, 38.0), flipped to the bottom, turned to 180 degrees
- moved C_1 23.0 mm to (58.9, 13.7)
- moved C_2 23.0 mm to (61.3, 10.9)
- moved L_1 23.0 mm to (66.7, 11.0)
- moved R_1 23.0 mm to (63.3, 15.1)
- moved U_1 23.0 mm to (61.2, 14.6)
- moved U$4 21.4 mm to (76.4, 13.3)
- moved U$5 21.4 mm to (73.9, 13.3)
- moved U$1 21.4 mm to (78.9, 13.3)
- moved R3 19.8 mm to (30.1, 27.6), turned to 270 degrees
- moved U$2 18.8 mm to (4.40, 21.2), turned to 270 degrees
- moved C3 16.2 mm to (61.6, 33.2)
- moved C4 16.2 mm to (61.3, 37.2)
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Connections:
- removed net N$13: R7.2, U1.3
- net N$12: now also U1.3; no longer R7.1
Routing:
- net 3.3V: track 31.5 -> 15.7 mm
- net N$24: track 2.70 -> 15.7 mm
- net N$12: track 2.01 -> 14.0 mm
- net 24V: track 11.7 -> 0.00 mm
- net N$13: track 11.5 -> 0.00 mm
- net N$17: track 21.0 -> 13.9 mm
- net N$23: track 3.21 -> 0.00 mm
- net N$21: track 3.21 -> 0.00 mm
- net N$22: track 2.45 -> 0.00 mm
- net N$16: track 2.30 -> 2.94 mm
- net N$15: track 14.8 -> 14.3 mm
Other:
- board size 132.6 x 103.3 mm -> 213.7 x 132 mm

Commit message: save?
Parts:
- moved U$3 23.3 mm to (23.9, 23.5)
- moved F1 22.6 mm to (7.30, 39.1), turned to 180 degrees
- moved C7 22.2 mm to (19.4, 37.6), turned to 270 degrees
- moved U$2 18.4 mm to (1.50, 39.4)
- moved D3 14.9 mm to (20.8, 27.8), turned to 180 degrees
- moved R9 6.96 mm to (25.4, 30.4), turned to 180 degrees
- moved R10 3.98 mm to (25.4, 32.5), turned to 180 degrees
Routing:
- net N$2: track 9.16 -> 0.00 mm
- net N$11: track 6.31 -> 0.00 mm
- net N$1: track 3.42 -> 0.00 mm
Other:
- board size 213.7 x 132 mm -> 234 x 132 mm

Commit message: ordered
Parts:
- removed C3: 220µF, derek:CAPPR5-10X16
- removed U$1, U$4, U$5: TP-1502, derek:TP-1502
- removed U$6: 10k, derek:0603
- removed U3: ESP-WROOM-32, derek:ESP-WROOM-32
- C2: value 220µF -> 470µF; device derek:CAPPR5-10X16 -> derek:CAPPR5-10X20
- moved L_1 37.1 mm to (58.0, 47.1), turned to 90 degrees
- moved C_2 36.4 mm to (63.4, 47.2), turned to 180 degrees
- moved U$8 33.2 mm to (68.0, 48.0)
- moved U$10 32.2 mm to (68.0, 46.0)
- moved C_1 31.4 mm to (66.0, 44.3), turned to 90 degrees
- moved U_1 29.0 mm to (63.5, 43.5), turned to 270 degrees
- moved R_1 28.0 mm to (61.4, 43.0), turned to 270 degrees
- moved U$3 24.0 mm to (0.00, 26.0)
- moved C7 18.8 mm to (26.4, 20.2), turned to 0 degrees
- moved C6 17.2 mm to (65.3, 38.6), turned to 0 degrees
- moved R101 14.0 mm to (65.3, 32.1)
- moved R1 9.94 mm to (65.3, 29.9)
- moved D3 9.10 mm to (12.0, 30.1), turned to 270 degrees
- moved C1 5.17 mm to (51.9, 17.5)
- moved U$9 5.13 mm to (68.0, 44.0)
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Connections:
- removed net N$21: U$1.1, U3.10
- removed net N$22: U$6.1, U3.3
- removed net N$23: U$5.1, U3.12
- removed net N$24: U$4.1, U3.11
- net 24V: no longer C3.P$1
- net 3.3V: no longer U$6.2, U3.2
- net GND-ISO: no longer C3.P$2, U3.1, U3.15, U3.38, U3.GND
Routing:
- net N$24: track 15.7 -> 0.00 mm
- net N$2: track 0.00 -> 10.2 mm
- net N$11: track 0.00 -> 9.19 mm
- net 3.3V: track 15.7 -> 22.5 mm
- net N$1: track 0.00 -> 3.03 mm
Other:
- board size 234 x 132 mm -> 146.1 x 62.4 mm
