File: pwr.brd (EAGLE design)
At the start: 71 x 42 mm, 39 parts, among them Q1 IPD65R600C6, T1 750811647, U1 UCC28700, U2 TPS62177

Commit message: use this
Parts:
- C3: value EEU-ED2G470S -> 47µF
Changed lines of the file:
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@@
 <element name="L" library="derek" package="TP-1502" value="TP-1502" x="69" y="15" rot="R270"/>
 <element name="N" library="derek" package="TP-1502" value="TP-1502" x="69" y="27" rot="R270"/>
-<element name="C3" library="derek" package="CAPPR7.5-18X20" value="EEU-ED2G470S" x="45" y="33" rot="R180"/>
+<element name="C3" library="derek" package="CAPPR7.5-18X20" value="47µF" x="45" y="33" rot="R180">
+<attribute name="DATASHEET_URL" value="https://industrial.panasonic.com/cdbs/www-data/pdf/RDF0000/ABA0000C1258.pdf" x="45" y="33" size="1.778" layer="27" rot="R180" display="off"/>
+<attribute name="DIGIKEY_PART_NUMBER" value="P13546-ND" x="45" y="33" size="1.778" layer="27" rot="R180" display="off"/>
+<attribute name="MANUFACTURER" value="Panasonic Electronic Components" x="45" y="33" size="1.778" layer="27" rot="R180" display="off"/>
+<attribute name="PART_NUMBER" value="EEU-ED2G470S" x="45" y="33" size="1.778" layer="27" rot="R180" display="off"/>
+<attribute name="VALUE" value="47µF" x="45" y="33" size="1.778" layer="27" rot="R180" display="off"/>
+</element>
 <element name="24V" library="derek" package="TP-1502" value="TP-1502" x="2" y="7" locked="yes" rot="R90"/>
 <element name="GND" library="derek" package="TP-1502" value="TP-1502" x="2" y="9" locked="yes" rot="R90"/>
