File: led.brd (EAGLE design)
At the start: 100 x 80 mm, 22 parts, among them U1 TPS92513HV

Commit message: save
Parts:
- removed C1: GRM32ER71J106KA12L, derek:1210_280
- removed C2: GCM155R71H103KA55D, derek:0402
- removed C3: CC0805KRX7R9BB103, derek:CC0805KRX7R9BB103
- removed C4: CC0805KRX7R8BB104, derek:CC0805KRX7R8BB104
- removed C5: 08053C104KAT2A, derek:0805
- removed C6: GMK212B7105KG-T, derek:GMK212B7105KG-T
- removed R1: CRCW0402121KFKED, derek:CRCW0402121KFKED
- removed R2: CRCW04027K68FKED, derek:CRCW04027K68FKED
- removed R3, R5: CRCW04021K00FKED, derek:CRCW04021K00FKED
- removed R4: CRCW0402162KFKED, derek:CRCW0402162KFKED
- removed R6: CRM0805-FX-R510ELF, derek:CRM0805-FX-R510ELF
- added CBOOT, CBOOT1: 08053C104KAT2A, derek:0805
- added CCOMP, CCOMP1: CC0805KRX7R8BB104, derek:CC0805KRX7R8BB104
- added CIADJ, CIADJ1: CC0805KRX7R9BB103, derek:CC0805KRX7R9BB103
- added CIN, CIN1: GRM32ER71J106KA12L, derek:1210_280
- added CINX, CINX1: GCM155R71H103KA55D, derek:0402
- added COUT, COUT1: GMK212B7105KG-T, derek:GMK212B7105KG-T
- added D10, D11, D12, D13, D14: XPGWHT, derek:XLAMP-XPG
- added D8: PMEG6010CEH,115, derek:SOD-123F
- added D9: BAT54WSTR, derek:SOD-323
- added J2: (no value), derek:1X02
- added L2: 74408943220, derek:IND_WE-SPC
- added RIADJ, RIADJ1, RSENSE1, RSENSE2: CRCW04021K00FKED, derek:CRCW04021K00FKED
- added RSENSE, RSENSE3: CRM0805-FX-R510ELF, derek:CRM0805-FX-R510ELF
- added RUVLOB, RUVLOB1: CRCW04027K68FKED, derek:CRCW04027K68FKED
- added RUVLOT, RUVLOT1: CRCW0402121KFKED, derek:CRCW0402121KFKED
- added R_RT, R_RT1: CRCW0402162KFKED, derek:CRCW0402162KFKED
- added U2: TPS92513HV, derek:TPS92513
- moved D7 64.8 mm to (13.2, 32.0), turned to 342 degrees
- moved D6 52.5 mm to (21.2, 14.9), turned to 54 degrees
- moved D3 49.3 mm to (27.0, 45.0)
- moved U1 37.6 mm to (68.4, 13.3)
- moved D2 37.1 mm to (74.8, 26.1)
- moved D5 33.7 mm to (40.0, 17.2), turned to 126 degrees
- moved D4 32.3 mm to (43.6, 35.8), turned to 198 degrees
- moved L1 32.2 mm to (74.8, 19.5)
- moved D1 26.1 mm to (73.8, 15.4)
- moved J1 22.3 mm to (13.0, 7.01), turned to 90 degrees
Connections:
- removed net GND: C1.2, C2.2, C3.2, C4.2, D1.2, J1.1, R2.2, R3.2, R4.2, R6.2, U1.9, U1.GND
- new net 24V: CIN.1, CIN1.1, CINX.1, CINX1.1, D2.1, D8.1, J1.2, RUVLOT.1, RUVLOT1.1, U1.2, U2.2
- new net GND-ISO: CCOMP.2, CCOMP1.2, CIADJ.2, CIADJ1.2, CIN.2, CIN1.2, CINX.2, CINX1.2, D1.2, D10.GND, D10.P$1, D10.P$2, D10.P$3, D11.GND, D11.P$1, D11.P$2, D11.P$3, D12.GND, D12.P$1, D12.P$2, D12.P$3, D13.GND, D13.P$1, D13.P$2, D13.P$3, D14.GND, D14.P$1, D14.P$2, D14.P$3, D3.GND, D3.P$1, D3.P$2, D3.P$3, D4.GND, D4.P$1, D4.P$2, D4.P$3, D5.GND, D5.P$1, D5.P$2, D5.P$3, D6.GND, D6.P$1, D6.P$2, D6.P$3, D7.GND, D7.P$1, D7.P$2, D7.P$3, D9.2, J1.1, RIADJ.2, RIADJ1.2, RSENSE.2, RSENSE3.2, RUVLOB.2, RUVLOB1.2, R_RT.2, R_RT1.2, U1.9, U1.GND-ISO, U1.P$1, U1.P$10, U1.P$11, U1.P$12, U1.P$2, U1.P$3, U1.P$4, U1.P$5, U1.P$6, U1.P$7, U1.P$8, U1.P$9, U2.9, U2.GND-ISO, U2.P$1, U2.P$10, U2.P$11, U2.P$12, U2.P$2, U2.P$3, U2.P$4, U2.P$5, U2.P$6, U2.P$7, U2.P$8, U2.P$9
- new net N$1: RUVLOB1.1, RUVLOT1.2, U2.3
- new net N$16: CBOOT1.1, D9.1, L2.1, U2.10
- new net N$17: COUT1.2, D14.C, RSENSE2.1, RSENSE3.1
- new net N$18: COUT1.1, D10.A, D8.2, L2.2
- new net N$19: R_RT1.1, U2.5
- new net N$20: CCOMP1.1, U2.8
- new net N$21: CBOOT1.2, U2.1
- new net N$22: RSENSE2.2, U2.7
- new net N$23: D10.C, D11.A
- new net N$24: D11.C, D12.A
- new net N$25: D12.C, D13.A
- new net N$26: D13.C, D14.A
- new net PDIM1: J2.1, U1.4
- new net PDIM2: J2.2, U2.4
- net N$10: now also CBOOT.2; no longer C5.2
- net N$11: now also RSENSE1.2; no longer R5.2
- net N$2: now also CIADJ.1, RIADJ.1; no longer C3.1, R3.1
- net N$3: now also RUVLOB.1, RUVLOT.2; no longer R1.2, R2.1
- net N$4: now also CIADJ1.1, RIADJ1.1, U2.6; no longer C1.1, C2.1, D2.1, J1.2, R1.1, U1.2
- net N$5: now also CBOOT.1; no longer C5.1
- net N$6: now also COUT.2, RSENSE.1, RSENSE1.1; no longer C6.2, R5.1, R6.1
- net N$7: now also COUT.1; no longer C6.1
- net N$8: now also R_RT.1; no longer R4.1
- net N$9: now also CCOMP.1; no longer C4.1
Routing:
- net N$24: track 0.00 -> 27.1 mm
- net N$23: track 0.00 -> 26.9 mm
- net N$25: track 0.00 -> 26.1 mm
- net N$12: track 0.00 -> 25.7 mm
- net N$13: track 0.00 -> 24.4 mm
- net N$14: track 0.00 -> 22.9 mm
- net N$11: track 0.00 -> 6.55 mm
- net N$10: track 0.00 -> 4.11 mm
- net N$3: track 0.00 -> 3.93 mm
- net N$2: track 0.00 -> 3.62 mm
- net N$9: track 0.00 -> 2.53 mm
- net N$8: track 0.00 -> 1.71 mm
- added copper zone on layer 1, net 24V
- added copper zone on layer 1, net GND-ISO
- added copper zone on layer 16, net GND-ISO
- added copper zone on layer 1, net N$5
- added copper zone on layer 1, net N$6
- added copper zone on layer 1, net N$7
- removed copper zone on layer 1, net GND
Other:
- board size 100 x 80 mm -> 58 x 58 mm

Commit message: save
Parts:
- CCOMP, CCOMP1: device derek:CC0805KRX7R8BB104 -> derek:0805
- CIADJ, CIADJ1: device derek:CC0805KRX7R9BB103 -> derek:0805
- CIN, CIN1: device derek:1210_280 -> derek:1210
- COUT, COUT1: device derek:GMK212B7105KG-T -> derek:0805
- RIADJ, RIADJ1, RSENSE1, RSENSE2: device derek:CRCW04021K00FKED -> derek:0402
- RSENSE, RSENSE3: device derek:CRM0805-FX-R510ELF -> derek:0805
- RUVLOB, RUVLOB1: device derek:CRCW04027K68FKED -> derek:0402
- RUVLOT, RUVLOT1: device derek:CRCW0402121KFKED -> derek:0402
- R_RT, R_RT1: device derek:CRCW0402162KFKED -> derek:0402
- moved L2 52.2 mm to (21.3, 49.6), turned to 0 degrees
- moved COUT1 50.5 mm to (23.0, 43.9)
- moved R_RT1 50.0 mm to (12.4, 40.5), turned to 270 degrees
- moved D9 49.6 mm to (20.1, 45.7), turned to 0 degrees
- moved RUVLOB 49.6 mm to (33.9, 49.8), turned to 198 degrees
- moved RUVLOB1 49.3 mm to (9.30, 40.5)
- moved CIN1 49.3 mm to (5.90, 42.0)
- moved RUVLOT1 49.3 mm to (9.30, 43.1)
- moved U2 49.3 mm to (14.6, 43.0)
- moved CBOOT1 49.2 mm to (14.7, 46.5)
- moved R_RT 49.2 mm to (34.5, 47.8), turned to 198 degrees
- moved CINX1 49.1 mm to (8.20, 43.1)
- moved RSENSE2 48.7 mm to (22.1, 39.7)
- moved CCOMP1 48.7 mm to (20.3, 43.0)
- moved RSENSE3 48.7 mm to (22.1, 41.2)
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Connections:
- net 24V: now also D2.C, D8.C; no longer D2.1, D8.1
- net GND-ISO: now also D1.A, D9.A; no longer D1.2, D9.2
- net N$12: now also D3.A, D7.C; no longer D3.C, D4.A
- net N$16: now also D9.C; no longer D9.1
- net N$18: now also D8.A; no longer D8.2
- net N$5: now also D1.C; no longer D1.1
- net N$6: now also D3.C; no longer D7.C
- net N$7: now also D2.A, D4.A; no longer D2.2, D3.A
Routing:
- net GND-ISO: track 0.00 -> 59.5 mm
- net 24V: track 0.00 -> 51.8 mm
- net N$18: track 0.00 -> 28.4 mm
- net N$7: track 0.07 -> 25.9 mm
- net PDIM2: track 0.00 -> 23.7 mm, vias 0 -> 1
- net N$26: track 0.00 -> 22.8 mm
- net N$15: track 0.00 -> 21.5 mm
- net N$6: track 0.00 -> 17.2 mm
- net N$16: track 0.00 -> 13.2 mm
- net N$17: track 0.00 -> 13.0 mm
- net N$5: track 0.00 -> 9.77 mm
- net PDIM1: track 0.00 -> 7.96 mm, vias 0 -> 1
- net N$23: track 26.9 -> 33.9 mm, vias 0 -> 2
- net N$22: track 0.00 -> 6.03 mm
- net N$1: track 0.00 -> 4.98 mm
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- removed copper zone on layer 1, net 24V
- removed copper zone on layer 1, net GND-ISO
- removed copper zone on layer 1, net N$5
- removed copper zone on layer 1, net N$6
- removed copper zone on layer 1, net N$7
Other:
- outline, holes or cut-outs redrawn

Commit message: ordered
Parts:
- turned D10 to 90 degrees
- turned D11 to 18 degrees
- turned D12 to 306 degrees
- turned D13 to 234 degrees
- turned D14 to 162 degrees
- turned D3 to 90 degrees
- turned D4 to 18 degrees
- turned D5 to 306 degrees
- turned D6 to 234 degrees
- turned D7 to 162 degrees
- renumbered D9 to GND-ISO
Routing:
- net GND-ISO: track 59.5 -> 54.9 mm, vias 0 -> 5
- added copper zone on layer 1, net GND-ISO

Commit message: should be good to order parts
Parts:
- CBOOT, CBOOT1: value 08053C104KAT2A -> 0.1µF
- CCOMP, CCOMP1: value CC0805KRX7R8BB104 -> 0.1µF
- CIADJ, CIADJ1: value CC0805KRX7R9BB103 -> 10000pF
- CIN, CIN1: value GRM32ER71J106KA12L -> 10µF
- CINX, CINX1: value GCM155R71H103KA55D -> 10000pF
- COUT, COUT1: value GMK212B7105KG-T -> 1µF
- D1, GND-ISO: value BAT54WSTR -> BAT54WS-TP
- D10, D11, D12, D13, D14: value XPGWHT -> XPGWHT-L1-0000-00G51
- D3, D4, D5, D6, D7: value XPGWHT -> XPGWHT-L1-0000-00BE8
- L1, L2: value 74408943220 -> 22µH
- RIADJ, RIADJ1, RSENSE1, RSENSE2: value CRCW04021K00FKED -> 1k
- RSENSE, RSENSE3: value CRM0805-FX-R510ELF -> 0.51
- RUVLOB, RUVLOB1: value CRCW04027K68FKED -> 7.68k
- RUVLOT, RUVLOT1: value CRCW0402121KFKED -> 121k
- R_RT, R_RT1: value CRCW0402162KFKED -> 162k

Commit message: order this
Parts:
- removed GND-ISO: BAT54WS-TP, derek:SOD-323
- added CIN2, CIN3: 1µF, derek:1206
- added D9: PMEG6010CEH,115, derek:SOD-123F
- CIN, CIN1: value 10µF -> 1µF; device derek:1210 -> derek:1206
- D1: value BAT54WS-TP -> PMEG6010CEH,115; device derek:SOD-323 -> derek:SOD-123F
- L1, L2: value 22µH -> 33µH; device derek:IND_WE-SPC -> derek:SRN6045
- RIADJ, RIADJ1, RSENSE1: value 1k -> 976
- RSENSE2: value 1k -> 0.51; device derek:0402 -> derek:0805
- RSENSE3: value 0.51 -> 976; device derek:0805 -> derek:0402
- RUVLOB, RUVLOB1: value 7.68k -> 5.49k
- RUVLOT, RUVLOT1: value 121k -> 97.6k
- U1, U2: value TPS92513HV -> TPS92513
- moved RSENSE2 1.50 mm to (22.1, 41.2)
- moved RSENSE3 1.50 mm to (22.1, 39.7)
- renumbered R_RT to RT, R_RT1 to RT1
Connections:
- net 24V: now also CIN2.1, CIN3.1
- net GND-ISO: now also CIN2.2, CIN3.2, D9.A, RSENSE2.2; no longer GND-ISO.A, RSENSE3.2
- net N$16: now also D9.C; no longer GND-ISO.C
- net N$22: now also RSENSE3.2; no longer RSENSE2.2
Routing:
- net GND-ISO: track 54.9 -> 56.1 mm
- net N$5: track 9.77 -> 9.16 mm
- net N$16: track 13.2 -> 12.6 mm

Commit message: save
Parts:
- moved D9 0.36 mm to (19.8, 45.5)
Routing:
- net GND-ISO: track 56.1 -> 46.8 mm
- net N$13: track 28.6 -> 23.1 mm, vias 2 -> 0
- net N$23: track 33.9 -> 28.7 mm
- net N$24: track 28.5 -> 24.6 mm
- net N$18: track 28.8 -> 30.0 mm
Other:
- outline, holes or cut-outs redrawn

Commit message: save
Parts:
- removed CBOOT, CBOOT1, CCOMP, CCOMP1: 0.1µF, derek:0805
- removed CIADJ, CIADJ1: 10000pF, derek:0805
- removed CIN, CIN1, CIN2, CIN3: 1µF, derek:1206
- removed CINX, CINX1: 10000pF, derek:0402
- removed COUT, COUT1: 1µF, derek:0805
- removed D10, D11, D12, D13, D14: XPGWHT-L1-0000-00G51, derek:XLAMP-XPG
- removed D8, D9: PMEG6010CEH,115, derek:SOD-123F
- removed J1, J2: (no value), derek:1X02
- removed L2: 33µH, derek:SRN6045
- removed RIADJ, RIADJ1, RSENSE1, RSENSE3: 976, derek:0402
- removed RSENSE, RSENSE2: 0.51, derek:0805
- removed RT, RT1: 162k, derek:0402
- removed RUVLOB, RUVLOB1: 5.49k, derek:0402
- removed RUVLOT, RUVLOT1: 97.6k, derek:0402
- removed U2: TPS92513, derek:TPS92513
- added C1, C2, C46, C48: 1µF, derek:1206
- added C3, C50: 10000pF, derek:0402
- added C4, C52: 470pF, derek:0603
- added C5, C54: 0.01μF, derek:0805
- added C56, C6: 0.1µF, derek:0603
- added C58, C7: 0.1µF, derek:0805
- added C60, C8: 1µF, derek:0805
- added D46, D48: PMEG6010CEH,115, derek:SOD-123F
- added D54, D55, D56, D57, D58: XPGWHT-L1-0000-00G51, derek:XLAMP-XPG
- added J45: (no value), derek:1X07_NO_SILK
- added L46: 33µH, derek:SRN6045
- added R1, R47: 97.6k, derek:0402
- added R2, R48: 5.49k, derek:0402
- added R3, R50: 162k, derek:0402
- added R4, R52: 4.02k, derek:0603
- added R5, R54: 976, derek:0402
- added R56, R6: 0.51, derek:0805
- added U46: TPS92513, derek:TPS92513
- moved U1 40.0 mm to (75.3, 60.3), turned to 270 degrees
- moved D1 40.0 mm to (71.2, 69.8), turned to 0 degrees
- moved L1 39.7 mm to (78.1, 68.3), turned to 90 degrees
- moved D2 38.8 mm to (79.0, 63.6), turned to 0 degrees
- moved D4 17.0 mm to (38.3, 19.7), turned to 306 degrees
- moved D5 17.0 mm to (23.0, 17.3), turned to 234 degrees
- moved D3 17.0 mm to (40.7, 34.9), turned to 18 degrees
- moved D6 17.0 mm to (16.0, 31.1), turned to 162 degrees
- moved D7 17.0 mm to (27.0, 42.0), turned to 90 degrees
Connections:
- removed net N$12 (its old number): D3.A, D7.C
- removed net N$2: CIADJ.1, RIADJ.1, U1.6
- removed net N$4: CIADJ1.1, RIADJ1.1, U2.6
- new net CLK: C4.2, C52.2, J45.1
- new net IADJ1: C5.1, J45.2, U1.6
- new net IADJ2: C54.1, J45.4, U46.6
- new net N$13: D3.C, D4.A
- new net N$34: C4.1, R4.1
- new net N$36: C52.1, R52.1
- net 24V: now also C1.1, C2.1, C3.1, C46.1, C48.1, C50.1, D1.C, D46.C, J45.7, R1.1, R47.1, U46.2; no longer CIN.1, CIN1.1, CIN2.1, CIN3.1, CINX.1, CINX1.1, D2.C, D8.C, J1.2, RUVLOT.1, RUVLOT1.1, U2.2
- net GND-ISO: now also C1.2, C2.2, C3.2, C46.2, C48.2, C5.2, C50.2, C54.2, C58.2, C7.2, D2.A, D48.A, D54.GND, D54.P$1, D54.P$2, D54.P$3, D55.GND, D55.P$1, D55.P$2, D55.P$3, D56.GND, D56.P$1, D56.P$2, D56.P$3, D57.GND, D57.P$1, D57.P$2, D57.P$3, D58.GND, D58.P$1, D58.P$2, D58.P$3, J45.6, R2.2, R3.2, R48.2, R50.2, R56.2, R6.2, U46.9, U46.GND-ISO, U46.P$1, U46.P$10, U46.P$11, U46.P$12, U46.P$2, U46.P$3, U46.P$4, U46.P$5, U46.P$6, U46.P$7, U46.P$8, U46.P$9; no longer CCOMP.2, CCOMP1.2, CIADJ.2, CIADJ1.2, CIN.2, CIN1.2, CIN2.2, CIN3.2, CINX.2, CINX1.2, D1.A, D10.GND, D10.P$1, D10.P$2, D10.P$3, D11.GND, D11.P$1, D11.P$2, D11.P$3, D12.GND, D12.P$1, D12.P$2, D12.P$3, D13.GND, D13.P$1, D13.P$2, D13.P$3, D14.GND, D14.P$1, D14.P$2, D14.P$3, D9.A, J1.1, RIADJ.2, RIADJ1.2, RSENSE.2, RSENSE2.2, RT.2, RT1.2, RUVLOB.2, RUVLOB1.2, U2.9, U2.GND-ISO, U2.P$1, U2.P$10, U2.P$11, U2.P$12, U2.P$2, U2.P$3, U2.P$4, U2.P$5, U2.P$6, U2.P$7, U2.P$8, U2.P$9
- net N$1: now also R47.2, R48.1, U46.3; no longer RUVLOB1.1, RUVLOT1.2, U2.3
- net N$10: now also C6.2; no longer CBOOT.2
- net N$11: now also R5.2; no longer RSENSE1.2
- net N$16: now also C56.1, D48.C, L46.1, U46.10; no longer CBOOT1.1, D9.C, L2.1, U2.10
- net N$17: now also C60.2, D58.C, R54.1, R56.1; no longer COUT1.2, D14.C, RSENSE2.1, RSENSE3.1
- net N$18: now also C60.1, D46.A, D54.A, L46.2; no longer COUT1.1, D10.A, D8.A, L2.2
- net N$19: now also R50.1, R52.2, U46.5; no longer RT1.1, U2.5
- net N$20: now also C58.1, U46.8; no longer CCOMP1.1, U2.8
- net N$21: now also C56.2, U46.1; no longer CBOOT1.2, U2.1
- net N$22: now also R54.2, U46.7; no longer RSENSE3.2, U2.7
- net N$23: now also D54.C, D55.A; no longer D10.C, D11.A
- net N$24: now also D55.C, D56.A; no longer D11.C, D12.A
- net N$25: now also D56.C, D57.A; no longer D12.C, D13.A
- net N$26: now also D57.C, D58.A; no longer D13.C, D14.A
- net N$3: now also R1.2, R2.1; no longer RUVLOB.1, RUVLOT.2
- net N$5: now also C6.1, D2.C; no longer CBOOT.1, D1.C
- net N$6: now also C8.2, D7.C, R5.1, R6.1; no longer COUT.2, D3.C, RSENSE.1, RSENSE1.1
- net N$7: now also C8.1, D1.A, D3.A; no longer COUT.1, D2.A, D4.A
- net N$8: now also R3.1, R4.2; no longer RT.1
- net N$9: now also C7.1; no longer CCOMP.1
- net PDIM1: now also J45.3; no longer J2.1
- net PDIM2: now also J45.5, U46.4; no longer J2.2, U2.4
Routing:
- net 24V: track 51.9 -> 1.83 mm
- net GND-ISO: track 46.8 -> 0.00 mm, vias 5 -> 34
- net N$18: track 30.0 -> 0.00 mm
- net N$23: track 28.7 -> 0.00 mm, vias 2 -> 0
- net N$7: track 25.6 -> 0.00 mm
- net N$24: track 24.6 -> 0.00 mm
- net N$25: track 23.9 -> 0.00 mm
- net PDIM2: track 23.7 -> 0.00 mm, vias 1 -> 0
- net N$14: track 23.1 -> 0.00 mm
- net N$26: track 22.8 -> 0.00 mm
- net N$12 (its old number): track 22.7 -> 0.00 mm
- net N$15: track 22.3 -> 0.00 mm
- net N$12: track 21.5 -> 0.00 mm
- net N$6: track 17.2 -> 0.00 mm
- net N$17: track 13.0 -> 0.00 mm
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- added copper zone on layer 1, net 24V
- added copper zone on layer 1, net N$5
- added copper zone on layer 1, net N$6
- added copper zone on layer 1, net N$7
