File: led.brd (EAGLE design)
At the start: 58 x 58 mm, 47 parts, among them U1 TPS92513, U46 TPS92513

Commit message: save
Parts:
- removed C46, C48: 1µF, derek:1206
- removed C50: 10000pF, derek:0402
- removed C52: 470pF, derek:0603
- removed C54: 0.01μF, derek:0805
- removed C56: 0.1µF, derek:0603
- removed C58: 0.1µF, derek:0805
- removed C60: 1µF, derek:0805
- removed D46, D48: PMEG6010CEH,115, derek:SOD-123F
- removed D54, D55, D56, D57, D58: XPGWHT-L1-0000-00G51, derek:XLAMP-XPG
- removed L46: 33µH, derek:SRN6045
- removed R47: 97.6k, derek:0402
- removed R48: 5.49k, derek:0402
- removed R50: 162k, derek:0402
- removed R52: 4.02k, derek:0603
- removed R54: 976, derek:0402
- removed R56: 0.51, derek:0805
- removed U46: TPS92513, derek:TPS92513
- moved C1 64.2 mm to (71.0, 64.0), turned to 0 degrees
- moved C2 0.30 mm to (71.0, 66.1)
- moved R5 0.20 mm to (82.2, 59.7)
- moved R6 0.20 mm to (82.8, 63.6)
- moved C8 0.18 mm to (83.6, 69.0)
- moved D2 0.10 mm to (79.0, 63.6)
- moved C3 0.07 mm to (71.7, 61.9)
Connections:
- removed net N$1: R47.2, R48.1, U46.3
- removed net N$16: C56.1, D48.C, L46.1, U46.10
- removed net N$17: C60.2, D58.C, R54.1, R56.1
- removed net N$18: C60.1, D46.A, D54.A, L46.2
- removed net N$19: R50.1, R52.2, U46.5
- removed net N$20: C58.1, U46.8
- removed net N$21: C56.2, U46.1
- removed net N$22: R54.2, U46.7
- removed net N$23: D54.C, D55.A
- removed net N$24: D55.C, D56.A
- removed net N$25: D56.C, D57.A
- removed net N$26: D57.C, D58.A
- removed net N$36: C52.1, R52.1
- net 24V: no longer C46.1, C48.1, C50.1, D46.C, R47.1, U46.2
- net CLK: no longer C52.2
- net GND-ISO: no longer C46.2, C48.2, C50.2, C54.2, C58.2, D48.A, D54.GND, D54.P$1, D54.P$2, D54.P$3, D55.GND, D55.P$1, D55.P$2, D55.P$3, D56.GND, D56.P$1, D56.P$2, D56.P$3, D57.GND, D57.P$1, D57.P$2, D57.P$3, D58.GND, D58.P$1, D58.P$2, D58.P$3, R48.2, R50.2, R56.2, U46.9, U46.GND-ISO, U46.P$1, U46.P$10, U46.P$11, U46.P$12, U46.P$2, U46.P$3, U46.P$4, U46.P$5, U46.P$6, U46.P$7, U46.P$8, U46.P$9
- net IADJ2: no longer C54.1, U46.6
- net PDIM2: no longer U46.4

Commit message: save
Parts:
- added C10: 10000pF, derek:0402
- added C11: 0.01μF, derek:0805
- added C12: 0.1µF, derek:0805
- added C13: 0.1µF, derek:0603
- added C14: 1µF, derek:0805
- added C15, C9: 1µF, derek:1206
- added C16: 470pF, derek:0603
- added D10, D11, D12, D13, D14: XPGWHT-L1-0000-00BE8, derek:XLAMP-XPG
- added D8, D9: PMEG6010CEH,115, derek:SOD-123F
- added L2: 33µH, derek:SRN6045
- added R10: 976, derek:0402
- added R11: 0.51, derek:0805
- added R12: 4.02k, derek:0603
- added R7: 97.6k, derek:0402
- added R8: 5.49k, derek:0402
- added R9: 162k, derek:0402
- added U2: TPS92513, derek:TPS92513
- moved D1 10.4 mm to (67.7, 60.0), turned to 54 degrees
- moved C2 8.51 mm to (70.6, 57.6), turned to 54 degrees
- moved R2 8.34 mm to (75.4, 53.1), turned to 324 degrees
- moved R1 8.17 mm to (74.1, 54.0), turned to 324 degrees
- moved C8 8.03 mm to (75.6, 69.6), turned to 324 degrees
- moved C1 7.72 mm to (72.3, 56.4), turned to 54 degrees
- moved R3 7.38 mm to (79.7, 53.3), turned to 324 degrees
- moved C4 6.78 mm to (80.9, 54.2), turned to 324 degrees
- moved C3 6.74 mm to (74.4, 55.7), turned to 144 degrees
- moved L1 6.32 mm to (72.9, 64.6), turned to 144 degrees
- moved R4 6.00 mm to (78.8, 54.8), turned to 234 degrees
- moved C5 4.15 mm to (80.8, 57.2), turned to 234 degrees
- moved C6 3.95 mm to (75.5, 59.0), turned to 234 degrees
- moved R6 3.91 mm to (79.5, 65.7), turned to 234 degrees
- moved U1 3.59 mm to (77.8, 57.7), turned to 324 degrees
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Connections:
- new net N$1: R7.2, R8.1, U2.3
- new net N$16: C13.1, D9.C, L2.1, U2.10
- new net N$17: R12.2, R9.1, U2.5
- new net N$18: C12.1, U2.8
- new net N$19: C13.2, U2.1
- new net N$2: D11.C, D12.A
- new net N$20: R10.2, U2.7
- new net N$21: D12.C, D13.A
- new net N$22: D13.C, D14.A
- new net N$23: C14.1, D11.A, D8.A, L2.2
- new net N$25: C16.1, R12.1
- new net N$4: C14.2, D10.C, R10.1, R11.1
- net 24V: now also C10.1, C15.1, C9.1, D8.C, R7.1, U2.2
- net CLK: now also C16.2
- net GND-ISO: now also C10.2, C11.2, C12.2, C15.2, C9.2, D10.GND, D10.P$1, D10.P$2, D10.P$3, D11.GND, D11.P$1, D11.P$2, D11.P$3, D12.GND, D12.P$1, D12.P$2, D12.P$3, D13.GND, D13.P$1, D13.P$2, D13.P$3, D14.GND, D14.P$1, D14.P$2, D14.P$3, D9.A, R11.2, R8.2, R9.2, U2.9, U2.GND-ISO, U2.P$1, U2.P$10, U2.P$11, U2.P$12, U2.P$2, U2.P$3, U2.P$4, U2.P$5, U2.P$6, U2.P$7, U2.P$8, U2.P$9
- net IADJ2: now also C11.1, U2.6
- net PDIM2: now also U2.4
Routing:
- net N$20: track 0.00 -> 4.94 mm
- net N$1: track 0.00 -> 4.44 mm
- net N$18: track 0.00 -> 3.11 mm
- net N$17: track 0.00 -> 2.78 mm
- net N$19: track 0.00 -> 2.42 mm
- net 24V: track 1.82 -> 3.63 mm
- net IADJ2: track 0.00 -> 1.74 mm
- net N$25: track 0.00 -> 1.35 mm
- added copper zone on layer 1, net N$16
- added copper zone on layer 1, net N$23
- added copper zone on layer 1, net N$4

Commit message: save
Parts:
- moved C14 87.8 mm to (32.7, 11.9), turned to 180 degrees
- moved R11 87.0 mm to (27.3, 12.7), turned to 90 degrees
- moved R10 86.5 mm to (23.4, 13.3), turned to 90 degrees
- moved C12 85.3 mm to (24.5, 15.2), turned to 0 degrees
- moved D9 84.6 mm to (27.3, 16.6), turned to 270 degrees
- moved L2 84.3 mm to (31.9, 17.5), turned to 0 degrees
- moved C11 82.9 mm to (21.2, 18.9), turned to 90 degrees
- moved U2 82.2 mm to (24.0, 20.2), turned to 180 degrees
- moved C13 82.1 mm to (26.6, 20.5), turned to 90 degrees
- moved C16 81.5 mm to (19.3, 21.2), turned to 180 degrees
- moved R12 81.1 mm to (21.4, 21.9), turned to 90 degrees
- moved R9 80.6 mm to (19.9, 22.6), turned to 180 degrees
- moved D8 80.2 mm to (33.4, 24.3), turned to 270 degrees
- moved C10 80.0 mm to (25.6, 23.8), turned to 0 degrees
- moved C9 79.8 mm to (29.7, 24.5), turned to 270 degrees
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Connections:
- new net N$24: D10.A, D14.C
- new net N$26: C14.2, R10.1, R11.1
- new net N$27: D10.C
- net N$23: no longer D11.A
- net N$4: now also D11.A; no longer C14.2, D10.C, R10.1, R11.1
Routing:
- net N$7: track 0.00 -> 49.2 mm
- net N$24: track 0.00 -> 32.8 mm
- net N$12: track 0.00 -> 31.6 mm
- net N$22: track 0.00 -> 30.8 mm
- net N$15: track 0.00 -> 29.5 mm
- net N$4: track 0.00 -> 19.4 mm
- net N$6: track 0.00 -> 4.34 mm
- added copper zone on layer 1, net N$26
- removed copper zone on layer 1, net N$4

Commit message: sent
Parts:
- moved J45 36.2 mm to (12.5, 32.1), flipped to the bottom
- moved C8 21.2 mm to (40.0, 32.9), turned to 180 degrees
- moved D1 21.2 mm to (40.7, 45.3), turned to 270 degrees
- moved C2 15.9 mm to (37.0, 45.5), turned to 270 degrees
- moved L1 15.1 mm to (39.2, 38.4), turned to 0 degrees
- moved R2 13.8 mm to (30.4, 46.4), turned to 180 degrees
- moved R1 13.6 mm to (32.0, 46.4), turned to 180 degrees
- moved C1 13.4 mm to (34.9, 45.5), turned to 270 degrees
- moved R6 13.1 mm to (34.5, 33.7), turned to 90 degrees
- moved R3 12.3 mm to (27.1, 43.6), turned to 180 degrees
- moved C4 11.5 mm to (26.6, 42.2), turned to 180 degrees
- moved R5 10.8 mm to (30.6, 34.3), turned to 90 degrees
- moved C3 10.7 mm to (32.9, 44.8), turned to 0 degrees
- moved R4 9.00 mm to (28.7, 42.9), turned to 90 degrees
- moved D2 6.94 mm to (34.6, 37.6), turned to 270 degrees
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Connections:
- removed net N$21: D12.C, D13.A
- removed net N$4: D11.A
- net IADJ1: now also J45.5; no longer J45.2
- net IADJ2: now also J45.2; no longer J45.4
- net N$23: now also D12.C
- net N$26: now also D13.A
- net N$27: now also D11.A
- net N$6: now also D3.A; no longer D7.C
- net N$7: now also D7.C; no longer D3.A
- net PDIM1: now also J45.4; no longer J45.3
- net PDIM2: now also J45.3; no longer J45.5
Routing:
- net 24V: track 3.63 -> 57.0 mm, vias 0 -> 1
- net N$27: track 0.00 -> 34.2 mm
- net CLK: track 0.00 -> 32.3 mm
- net N$2: track 0.00 -> 31.5 mm
- net N$26: track 0.00 -> 30.2 mm
- net N$14: track 0.00 -> 29.5 mm, vias 0 -> 2
- net N$13: track 0.00 -> 28.6 mm
- net N$6: track 4.34 -> 30.1 mm
- net PDIM1: track 0.00 -> 23.5 mm, vias 0 -> 1
- net N$4: track 19.4 -> 0.00 mm
- net IADJ2: track 1.74 -> 20.3 mm, vias 0 -> 1
- net N$7: track 49.2 -> 34.1 mm
- net PDIM2: track 0.00 -> 13.2 mm
- net IADJ1: track 1.74 -> 12.6 mm
- net N$23: track 0.00 -> 6.25 mm
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
Commit message: save
Parts:
- removed C10: 10000pF, derek:0402
- removed C11: 0.01μF, derek:0805
- removed C12, C7: 0.1µF, derek:0805
- removed C13, C6: 0.1µF, derek:0603
- removed C14, C8: 1µF, derek:0805
- removed C15, C9: 1µF, derek:1206
- removed C16: 470pF, derek:0603
- removed D1, D2, D8, D9: PMEG6010CEH,115, derek:SOD-123F
- removed D10, D11, D12, D13, D14, D3, D4, D5, D6, D7: XPGWHT-L1-0000-00BE8, derek:XLAMP-XPG
- removed J45: (no value), derek:1X07_NO_SILK
- removed L1, L2: 33µH, derek:SRN6045
- removed R1, R7: 97.6k, derek:0402
- removed R10, R5: 976, derek:0402
- removed R11, R6: 0.51, derek:0805
- removed R12, R4: 4.02k, derek:0603
- removed R2, R8: 5.49k, derek:0402
- removed R3, R9: 162k, derek:0402
- removed U1, U2: TPS92513, derek:TPS92513
- added C+, C-, W+, W-: TP-1502, derek:TP-1502
- added W1, W2, W3, W4, W5: XPGWHT-L1-0000-00BE8, derek:XLAMP-XPG
- C1, C2: value 1µF -> XPGWHT-L1-0000-00BE8; device derek:1206 -> derek:XLAMP-XPG
- C3: value 10000pF -> XPGWHT-L1-0000-00BE8; device derek:0402 -> derek:XLAMP-XPG
- C4: value 470pF -> XPGWHT-L1-0000-00BE8; device derek:0603 -> derek:XLAMP-XPG
- C5: value 0.01μF -> XPGWHT-L1-0000-00BE8; device derek:0805 -> derek:XLAMP-XPG
- moved C3 42.1 mm to (9.74, 9.66), turned to 234 degrees
- moved C2 40.1 mm to (25.0, 7.31), turned to 306 degrees
- moved C4 26.0 mm to (7.25, 24.9), turned to 162 degrees
- moved C1 24.6 mm to (32.0, 21.1), turned to 18 degrees
- moved C5 10.9 mm to (21.0, 32.0)
Connections:
- removed net 24V: C1.1, C10.1, C15.1, C2.1, C3.1, C9.1, D1.C, D8.C, J45.7, R1.1, R7.1, U1.2, U2.2
- removed net CLK: C16.2, C4.2, J45.1
- removed net IADJ1: C5.1, J45.5, U1.6
- removed net IADJ2: C11.1, J45.2, U2.6
- removed net N$10: C6.2, U1.1
- removed net N$11: R5.2, U1.7
- removed net N$16: C13.1, D9.C, L2.1, U2.10
- removed net N$17: R12.2, R9.1, U2.5
- removed net N$18: C12.1, U2.8
- removed net N$19: C13.2, U2.1
- removed net N$20: R10.2, U2.7
- removed net N$23: C14.1, D12.C, D8.A, L2.2
- removed net N$25: C16.1, R12.1
- removed net N$26: C14.2, D13.A, R10.1, R11.1
- removed net N$27: D10.C, D11.A
- removed net N$34: C4.1, R4.1
- removed net N$5: C6.1, D2.C, L1.1, U1.10
- removed net N$6: C8.2, D3.A, R5.1, R6.1
- removed net N$7: C8.1, D1.A, D7.C, L1.2
- removed net N$8: R3.1, R4.2, U1.5
- removed net N$9: C7.1, U1.8
- removed net PDIM1: J45.4, U1.4
- removed net PDIM2: J45.3, U2.4
- new net N$30: W+.1, W1.A
- new net N$31: W-.1, W5.C
- new net N$4: C-.1, C5.C
- net GND-ISO: now also C1.GND, C1.P$1, C1.P$2, C1.P$3, C2.GND, C2.P$1, C2.P$2, C2.P$3, C3.GND, C3.P$1, C3.P$2, C3.P$3, C4.GND, C4.P$1, C4.P$2, C4.P$3, C5.GND, C5.P$1, C5.P$2, C5.P$3, W1.GND, W1.P$1, W1.P$2, W1.P$3, W2.GND, W2.P$1, W2.P$2, W2.P$3, W3.GND, W3.P$1, W3.P$2, W3.P$3, W4.GND, W4.P$1, W4.P$2, W4.P$3, W5.GND, W5.P$1, W5.P$2, W5.P$3; no longer C1.2, C10.2, C11.2, C12.2, C15.2, C2.2, C3.2, C5.2, C7.2, C9.2, D10.GND, D10.P$1, D10.P$2, D10.P$3, D11.GND, D11.P$1, D11.P$2, D11.P$3, D12.GND, D12.P$1, D12.P$2, D12.P$3, D13.GND, D13.P$1, D13.P$2, D13.P$3, D14.GND, D14.P$1, D14.P$2, D14.P$3, D2.A, D3.GND, D3.P$1, D3.P$2, D3.P$3, D4.GND, D4.P$1, D4.P$2, D4.P$3, D5.GND, D5.P$1, D5.P$2, D5.P$3, D6.GND, D6.P$1, D6.P$2, D6.P$3, D7.GND, D7.P$1, D7.P$2, D7.P$3, D9.A, J45.6, R11.2, R2.2, R3.2, R6.2, R8.2, R9.2, U1.9, U1.GND-ISO, U1.P$1, U1.P$10, U1.P$11, U1.P$12, U1.P$2, U1.P$3, U1.P$4, U1.P$5, U1.P$6, U1.P$7, U1.P$8, U1.P$9, U2.9, U2.GND-ISO, U2.P$1, U2.P$10, U2.P$11, U2.P$12, U2.P$2, U2.P$3, U2.P$4, U2.P$5, U2.P$6, U2.P$7, U2.P$8, U2.P$9
- net N$1: now also C2.C, C3.A; no longer R7.2, R8.1, U2.3
- net N$12: now also W4.C, W5.A; no longer D6.C, D7.A
- net N$13: now also W1.C, W2.A; no longer D3.C, D4.A
- net N$14: now also W2.C, W3.A; no longer D4.C, D5.A
- net N$15: now also W3.C, W4.A; no longer D5.C, D6.A
- net N$2: now also C1.C, C2.A; no longer D11.C, D12.A
- net N$22: now also C3.C, C4.A; no longer D13.C, D14.A
- net N$24: now also C4.C, C5.A; no longer D10.A, D14.C
- net N$3: now also C+.1, C1.A; no longer R1.2, R2.1, U1.3
Routing:
- net 24V: track 57.0 -> 0.00 mm, vias 1 -> 0
- net N$24: track 35.2 -> 0.00 mm
- net N$12: track 34.3 -> 0.00 mm
- net N$27: track 34.2 -> 0.00 mm
- net N$7: track 34.1 -> 0.00 mm
- net CLK: track 32.3 -> 0.00 mm
- net N$2: track 31.5 -> 0.00 mm
- net N$22: track 30.8 -> 0.00 mm
- net N$26: track 30.2 -> 0.00 mm
- net N$6: track 30.1 -> 0.00 mm
- net N$14: track 29.5 -> 0.00 mm, vias 2 -> 0
- net N$15: track 29.5 -> 0.00 mm
- net N$13: track 28.6 -> 0.00 mm
- net PDIM1: track 23.5 -> 0.00 mm, vias 1 -> 0
- net IADJ2: track 20.3 -> 0.00 mm, vias 1 -> 0
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- removed copper zone on layer 1, net 24V
- removed copper zone on layer 1, net N$16
- removed copper zone on layer 1, net N$23
- removed copper zone on layer 1, net N$26
- removed copper zone on layer 1, net N$5
- removed copper zone on layer 1, net N$6
- removed copper zone on layer 1, net N$7
Other:
- board size 58 x 58 mm -> 38 x 38 mm

Commit message: save
Parts:
- moved C+ 9.70 mm to (22.0, 28.7)
- moved C- 9.70 mm to (20.0, 28.7)
- moved W+ 9.70 mm to (18.0, 28.7)
- moved W- 9.70 mm to (16.0, 28.7)
Changed lines of the file:
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@@
 <attribute name="VALUE" x="7.8296875" y="26.690165625" size="0.6096" layer="27" font="vector" ratio="20" rot="R162" align="top-center"/>
 </element>
-<element name="W+" library="derek" package="TP-1502" value="TP-1502" x="18" y="19" rot="MR0"/>
-<element name="W-" library="derek" package="TP-1502" value="TP-1502" x="16" y="19" rot="MR0"/>
-<element name="C+" library="derek" package="TP-1502" value="TP-1502" x="22" y="19" rot="MR0"/>
-<element name="C-" library="derek" package="TP-1502" value="TP-1502" x="20" y="19" rot="MR0"/>
+<element name="W+" library="derek" package="TP-1502" value="TP-1502" x="18" y="28.7" locked="yes" rot="MR0"/>
+<element name="W-" library="derek" package="TP-1502" value="TP-1502" x="16" y="28.7" locked="yes" rot="MR0"/>
+<element name="C+" library="derek" package="TP-1502" value="TP-1502" x="22" y="28.7" locked="yes" rot="MR0"/>
+<element name="C-" library="derek" package="TP-1502" value="TP-1502" x="20" y="28.7" locked="yes" rot="MR0"/>
 </elements>
 <signals>
@@
 <contactref element="W1" pad="A"/>
 <contactref element="W+" pad="1"/>
-<wire x1="18" y1="19" x2="32.077178125" y2="25.351921875" width="0" layer="19" extent="1-1"/>
+<wire x1="18" y1="28.7" x2="32.077178125" y2="25.351921875" width="0" layer="19" extent="1-1"/>
 </signal>
 <signal name="N$31">
 <contactref element="W5" pad="C"/>
 <contactref element="W-" pad="1"/>
-<wire x1="16" y1="19" x2="17" y2="30.6" width="0" layer="19" extent="1-1"/>
+<wire x1="16" y1="28.7" x2="17" y2="30.6" width="0" layer="19" extent="1-1"/>
 </signal>
 <signal name="N$1">
@@
 <contactref element="C1" pad="A"/>
 <contactref element="C+" pad="1"/>
-<wire x1="22" y1="19" x2="33.313278125" y2="21.547721875" width="0" layer="19" extent="1-1"/>
+<wire x1="22" y1="28.7" x2="33.313278125" y2="21.547721875" width="0" layer="19" extent="1-1"/>
 </signal>
 <signal name="N$4">
 <contactref element="C5" pad="C"/>
 <contactref element="C-" pad="1"/>
-<wire x1="20" y1="19" x2="21" y2="30.6" width="0" layer="19" extent="1-1"/>
+<wire x1="20" y1="28.7" x2="21" y2="30.6" width="0" layer="19" extent="1-1"/>
 </signal>
 </signals>

Commit message: ORDERED
Routing:
- net N$2: track 0.00 -> 23.6 mm
- net N$22: track 0.00 -> 22.6 mm
- net N$13: track 0.00 -> 22.4 mm
- net N$1: track 0.00 -> 21.5 mm
- net N$24: track 0.00 -> 20.8 mm
- net N$15: track 0.00 -> 20.6 mm
- net N$3: track 0.00 -> 20.3 mm
- net N$12: track 0.00 -> 20.0 mm
- net N$14: track 0.00 -> 19.9 mm
- net N$30: track 0.00 -> 18.7 mm
- net N$4: track 0.00 -> 2.31 mm
- net N$31: track 0.00 -> 2.31 mm
Changed lines of the file:
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@@
 <contactref element="W1" pad="C"/>
 <contactref element="W2" pad="A"/>
-<wire x1="29.082096875" y1="8.525675" x2="29.41421875" y2="24.486675" width="0" layer="19" extent="1-1"/>
+<wire x1="29.41421875" y1="24.486675" x2="28.2" y2="23.27245625" width="0.3048" layer="1"/>
+<wire x1="28.2" y1="23.27245625" x2="28.2" y2="15.9" width="0.3048" layer="1"/>
+<wire x1="28.2" y1="15.9" x2="32.6" y2="11.5" width="0.3048" layer="1"/>
+<wire x1="32.6" y1="11.5" x2="32.6" y2="8.6" width="0.3048" layer="1"/>
+<wire x1="32.6" y1="8.6" x2="31.7" y2="7.7" width="0.3048" layer="1"/>
+<wire x1="31.7" y1="7.7" x2="30.7" y2="7.7" width="0.3048" layer="1"/>
+<wire x1="30.7" y1="7.7" x2="29.874325" y2="8.525675" width="0.3048" layer="1"/>
+<wire x1="29.874325" y1="8.525675" x2="29.082096875" y2="8.525675" width="0.3048" layer="1"/>
 </signal>
 <signal name="N$14">
 <contactref element="W2" pad="C"/>
 <contactref element="W3" pad="A"/>
-<wire x1="12.1539" y1="6.174575" x2="27.4363" y2="10.790921875" width="0" layer="19" extent="1-1"/>
+<wire x1="27.4363" y1="10.790921875" x2="21.290921875" y2="10.790921875" width="0.3048" layer="1"/>
+<wire x1="21.290921875" y1="10.790921875" x2="14.8" y2="4.3" width="0.3048" layer="1"/>
+<wire x1="14.8" y1="4.3" x2="12.5" y2="4.3" width="0.3048" layer="1"/>
+<wire x1="12.5" y1="4.3" x2="11.9" y2="4.9" width="0.3048" layer="1"/>
+<wire x1="11.9" y1="4.9" x2="11.9" y2="5.920675" width="0.3048" layer="1"/>
+<wire x1="11.9" y1="5.920675" x2="12.1539" y2="6.174575" width="0.3048" layer="1"/>
 </signal>
 <signal name="N$15">
 <contactref element="W3" pad="C"/>
 <contactref element="W4" pad="A"/>
-<wire x1="13.799696875" y1="8.439821875" x2="4.68671875" y2="21.547721875" width="0" layer="19" extent="1-1"/>
+<wire x1="13.799696875" y1="8.439821875" x2="13.799696875" y2="12.300303125" width="0.3048" layer="1"/>
+<wire x1="13.799696875" y1="12.300303125" x2="9.5" y2="16.6" width="0.3048" layer="1"/>
+<wire x1="9.5" y1="16.6" x2="5.6" y2="16.6" width="0.3048" layer="1"/>
+<wire x1="5.6" y1="16.6" x2="2.9" y2="19.3" width="0.3048" layer="1"/>
+<wire x1="2.9" y1="19.3" x2="2.9" y2="19.761003125" width="0.3048" layer="1"/>
+<wire x1="2.9" y1="19.761003125" x2="4.68671875" y2="21.547721875" width="0.3048" layer="1"/>
 </signal>
 <signal name="GND-ISO">
@@
 <contactref element="W4" pad="C"/>
 <contactref element="W5" pad="A"/>
-<wire x1="7.349678125" y1="20.682475" x2="17" y2="33.4" width="0" layer="19" extent="1-1"/>
+<wire x1="7.349678125" y1="20.682475" x2="13" y2="26.332796875" width="0.3048" layer="1"/>
+<wire x1="13" y1="26.332796875" x2="13" y2="32.3" width="0.3048" layer="1"/>
+<wire x1="13" y1="32.3" x2="15.5" y2="34.8" width="0.3048" layer="1"/>
+<wire x1="15.5" y1="34.8" x2="16.3" y2="34.8" width="0.3048" layer="1"/>
+<wire x1="16.3" y1="34.8" x2="17" y2="34.1" width="0.3048" layer="1"/>
+<wire x1="17" y1="34.1" x2="17" y2="33.4" width="0.3048" layer="1"/>
 </signal>
 <signal name="N$2">
 <contactref element="C2" pad="A"/>
 <contactref element="C1" pad="C"/>
-<wire x1="25.846096875" y1="6.174575" x2="30.65031875" y2="20.682475" width="0" layer="19" extent="1-1"/>
+<wire x1="30.65031875" y1="20.682475" x2="29.2" y2="19.23215625" width="0.3048" layer="1"/>
+<wire x1="29.2" y1="19.23215625" x2="29.2" y2="16.4" width="0.3048" layer="1"/>
+<wire x1="29.2" y1="16.4" x2="33.6" y2="12" width="0.3048" layer="1"/>
+<wire x1="33.6" y1="12" x2="33.6" y2="8" width="0.3048" layer="1"/>
+<wire x1="33.6" y1="8" x2="31.774575" y2="6.174575" width="0.3048" layer="1"/>
+<wire x1="31.774575" y1="6.174575" x2="25.846096875" y2="6.174575" width="0.3048" layer="1"/>
 </signal>
 <signal name="N$22">
 <contactref element="C3" pad="C"/>
 <contactref element="C4" pad="A"/>
-<wire x1="10.563696875" y1="10.790921875" x2="5.92281875" y2="25.351921875" width="0" layer="19" extent="1-1"/>
+<wire x1="10.563696875" y1="10.790921875" x2="10.563696875" y2="13.336303125" width="0.3048" layer="1"/>
+<wire x1="10.563696875" y1="13.336303125" x2="8.8" y2="15.1" width="0.3048" layer="1"/>
+<wire x1="8.8" y1="15.1" x2="4.9" y2="15.1" width="0.3048" layer="1"/>
+<wire x1="4.9" y1="15.1" x2="1.3" y2="18.7" width="0.3048" layer="1"/>
+<wire x1="1.3" y1="18.7" x2="1.3" y2="20.729103125" width="0.3048" layer="1"/>
+<wire x1="1.3" y1="20.729103125" x2="5.92281875" y2="25.351921875" width="0.3048" layer="1"/>
 </signal>
 <signal name="N$24">
 <contactref element="C5" pad="A"/>
 <contactref element="C4" pad="C"/>
-<wire x1="8.585778125" y1="24.486675" x2="21" y2="33.4" width="0" layer="19" extent="1-1"/>
+<wire x1="8.585778125" y1="24.486675" x2="12" y2="27.900896875" width="0.3048" layer="1"/>
+<wire x1="12" y1="32.6" x2="15.2" y2="35.8" width="0.3048" layer="1"/>
+<wire x1="15.2" y1="35.8" x2="18.6" y2="35.8" width="0.3048" layer="1"/>
+<wire x1="18.6" y1="35.8" x2="21" y2="33.4" width="0.3048" layer="1"/>
+<wire x1="12" y1="27.900896875" x2="12" y2="32.6" width="0.3048" layer="1"/>
 </signal>
 <signal name="N$30">
 <contactref element="W1" pad="A"/>
 <contactref element="W+" pad="1"/>
-<wire x1="18" y1="28.7" x2="32.077178125" y2="25.351921875" width="0" layer="19" extent="1-1"/>
+<wire x1="18" y1="28.7" x2="20.6" y2="26.1" width="0.3048" layer="1"/>
+<wire x1="22.9" y1="26.1" x2="20.6" y2="26.1" width="0.3048" layer="1"/>
+<wire x1="32.077178125" y1="25.351921875" x2="32.077178125" y2="27.722821875" width="0.3048" layer="1"/>
+<wire x1="32.077178125" y1="27.722821875" x2="31.5" y2="28.3" width="0.3048" layer="1"/>
+<wire x1="31.5" y1="28.3" x2="25.1" y2="28.3" width="0.3048" layer="1"/>
+<wire x1="25.1" y1="28.3" x2="22.9" y2="26.1" width="0.3048" layer="1"/>
 </signal>
 <signal name="N$31">
 <contactref element="W5" pad="C"/>
 <contactref element="W-" pad="1"/>
-<wire x1="16" y1="28.7" x2="17" y2="30.6" width="0" layer="19" extent="1-1"/>
+<wire x1="16" y1="28.7" x2="16" y2="29.6" width="0.3048" layer="1"/>
+<wire x1="16" y1="29.6" x2="17" y2="30.6" width="0.3048" layer="1"/>
 </signal>
 <signal name="N$1">
 <contactref element="C2" pad="C"/>
 <contactref element="C3" pad="A"/>
-<wire x1="8.9179" y1="8.525675" x2="24.2003" y2="8.439821875" width="0" layer="19" extent="1-1"/>
+<wire x1="24.2003" y1="8.439821875" x2="20.439821875" y2="8.439821875" width="0.3048" layer="1"/>
+<wire x1="20.439821875" y1="8.439821875" x2="14.9" y2="2.9" width="0.3048" layer="1"/>
+<wire x1="14.9" y1="2.9" x2="11.8" y2="2.9" width="0.3048" layer="1"/>
+<wire x1="8.9179" y1="5.7821" x2="8.9179" y2="8.525675" width="0.3048" layer="1"/>
+<wire x1="11.8" y1="2.9" x2="8.9179" y2="5.7821" width="0.3048" layer="1"/>
 </signal>
 <signal name="N$3">
 <contactref element="C1" pad="A"/>
 <contactref element="C+" pad="1"/>
-<wire x1="22" y1="28.7" x2="33.313278125" y2="21.547721875" width="0" layer="19" extent="1-1"/>
+<wire x1="22" y1="28.7" x2="22.8" y2="29.5" width="0.3048" layer="1"/>
+<wire x1="22.8" y1="29.5" x2="32.7" y2="29.5" width="0.3048" layer="1"/>
+<wire x1="34.6" y1="27.6" x2="34.6" y2="22.8" width="0.3048" layer="1"/>
+<wire x1="34.6" y1="22.8" x2="33.347721875" y2="21.547721875" width="0.3048" layer="1"/>
+<wire x1="33.347721875" y1="21.547721875" x2="33.313278125" y2="21.547721875" width="0.3048" layer="1"/>
+<wire x1="32.7" y1="29.5" x2="34.6" y2="27.6" width="0.3048" layer="1"/>
 </signal>
 <signal name="N$4">
 <contactref element="C5" pad="C"/>
 <contactref element="C-" pad="1"/>
-<wire x1="20" y1="28.7" x2="21" y2="30.6" width="0" layer="19" extent="1-1"/>
+<wire x1="20" y1="28.7" x2="20" y2="29.6" width="0.3048" layer="1"/>
+<wire x1="20" y1="29.6" x2="21" y2="30.6" width="0.3048" layer="1"/>
 </signal>
 </signals>
