File: pwr.sch (EAGLE design)
At the start: 43 parts, among them Q1 IPD65R600E6, T1 750811647, U1 UCC28700

Commit message: save
Parts:
- removed U$5, U$6, U$7: TP-1502, derek:TP-1502
Connections:
- net 24V: no longer U$5.TP
- net GND-ISO: no longer U$6.TP, U$7.TP
Other:
- moved on the sheet: C_1, C_2, L_1, R_1, U$8, U_1

Commit message: getting close
Parts:
- added U2: ESP3212, derek:ESP3212
- C1: value DE1E3KX222MA4BL01 -> 2200pF; device derek:DE1E3KX222MA4BL01 -> derek:DE1E3KX222MA4BN01F
- C2, C3: value UHE1V221MPD6 -> 220µF
- C4, C5: value UMK316AB7475KL-T -> 4.7µF
- C6: value 08053C104KAT2A -> 0.1µF
- C7: value EEUED2G470 -> 47µF; device derek:EEUED2G470 -> derek:EEU-ED2G470
- C8: value 06035C104KAT2A -> 0.1µF
- C9: value GRM31CR61H225KA88L -> 2.2µF
- C_1: value C1608X5R1V225K080AC -> 2.2µF
- C_2: value GRM21BR60J226ME39L -> 22µF
- Q1: value IPD65R600E6 -> IPD65R600C6; device derek:IPD65R600E6 -> derek:IPD65R600C6
- R1, R101: value CRCW120610K0JNEA -> 10k
- R10, R9: value CSR1206FKR750 -> 0.75
- R11: value CRCW060319K6FKEA -> 19.6k
- R2: value CRCW120633R2FKEA -> 33.2; device derek:CRCW120633R2FKEA -> derek:CRCW121033R2FKEA
- R3: value CRCW12064R70JNEA -> 4.7
- R4: value CRCW060375K0FKEA -> 75k
- R5, R6: value CRCW08053M30JNEA -> 3.3M
- R7: value CRCW06030000Z0EA -> 0.0
- R8: value CRCW1206698RFKEA -> 698
- R_1: value CRCW0402100KFKED -> 100k

Commit message: pwr to osh
Parts:
- removed U2: ESP3212, derek:ESP3212
- L_1: value LPS4018-103MRBLPS4018-103MRB -> 10µH; device derek:LPS4018-103MRBLPS4018-103MRB -> derek:SDR0503-100ML
Changed lines of the file:
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@@
 <part name="C_1" library="derek" deviceset="C1608X5R1V225K080AC" device="" value="2.2µF"/>
 <part name="R_1" library="derek" deviceset="CRCW0402100KFKED" device="" value="100k"/>
-<part name="L_1" library="derek" deviceset="LPS4018-103MRB" device="LPS4018-103MRB"/>
+<part name="L_1" library="derek" deviceset="SDR0503-100ML" device="" value="10µH"/>
 <part name="C_2" library="derek" deviceset="GRM21BR60J226ME39L" device="" value="22µF"/>
 <part name="U$8" library="derek" deviceset="TP-1502" device=""/>
@@
 <part name="SUPPLY3" library="derek" deviceset="24V" device=""/>
 <part name="F1" library="derek" deviceset="37012000410" device=""/>
-<part name="U2" library="derek" deviceset="ESP3212" device=""/>
 </parts>
 <sheets>
@@
 <instance part="SUPPLY3" gate="G$1" x="302.26" y="63.5"/>
 <instance part="F1" gate="G$1" x="48.26" y="25.4"/>
-<instance part="U2" gate="G$1" x="332.74" y="-104.14"/>
 </instances>
 <busses>

Commit message: save
Parts:
- added U$1, U$4, U$5: TP-1502, derek:TP-1502
- added U3: ESP-WROOM-32, derek:ESP-WROOM-32
Connections:
- new net N$21: U$1.TP, U3.IO25
- new net N$23: U$5.TP, U3.IO27
- new net N$24: U$4.TP, U3.IO26
- net 3.3V: now also U3.3V3
- net GND: now also U1.GND
- net GND-ISO: now also U3.GND, U3.GND@1, U3.GND@15, U3.GND@38

Commit message: save
Connections:
- net N$14: now also D5.C; no longer D5.K
- net N$8: now also D4.C; no longer D4.K
Changed lines of the file:
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@@
 <segment>
 <pinref part="D2" gate="G$1" pin="C"/>
-<pinref part="D4" gate="G$1" pin="K"/>
+<pinref part="D4" gate="G$1" pin="C"/>
 <wire x1="142.24" y1="25.4" x2="142.24" y2="20.32" width="0.1524" layer="91"/>
 </segment>
@@
 <pinref part="R5" gate="G$1" pin="2"/>
 <wire x1="99.06" y1="-96.52" x2="101.6" y2="-96.52" width="0.1524" layer="91"/>
-<pinref part="D5" gate="G$1" pin="K"/>
+<pinref part="D5" gate="G$1" pin="C"/>
 <wire x1="99.06" y1="-96.52" x2="38.1" y2="-96.52" width="0.1524" layer="91"/>
 <wire x1="38.1" y1="-96.52" x2="38.1" y2="-91.44" width="0.1524" layer="91"/>
