File: pwr.sch (EAGLE design)
At the start: 44 parts, among them Q1 IPD65R600C6, T1 750811647, U1 UCC28700, U3 ESP-WROOM-32

Commit message: ordered
Parts:
- added U$6: 10k, derek:CRCW060310K0FKEA
Connections:
- new net N$22: U$6.1, U3.EN
- net 3.3V: now also U$6.2
Changed lines of the file:
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@@
 <part name="GND-ISO8" library="derek" deviceset="GND-ISO" device=""/>
 <part name="U$5" library="derek" deviceset="TP-1502" device=""/>
+<part name="U$6" library="derek" deviceset="CRCW060310K0FKEA" device="" value="10k"/>
 </parts>
 <sheets>
@@
 <instance part="GND-ISO8" gate="G$1" x="472.44" y="-68.58"/>
 <instance part="U$5" gate="A" x="429.26" y="-96.52"/>
+<instance part="U$6" gate="G$1" x="436.88" y="-45.72"/>
 </instances>
 <busses>
@@
 <wire x1="447.04" y1="-43.18" x2="426.72" y2="-43.18" width="0.1524" layer="91"/>
 <wire x1="426.72" y1="-43.18" x2="426.72" y2="-40.64" width="0.1524" layer="91"/>
+<pinref part="U$6" gate="G$1" pin="2"/>
+<wire x1="429.26" y1="-45.72" x2="426.72" y2="-45.72" width="0.1524" layer="91"/>
+<wire x1="426.72" y1="-45.72" x2="426.72" y2="-43.18" width="0.1524" layer="91"/>
+<junction x="426.72" y="-43.18"/>
 </segment>
 </net>
@@
 </segment>
 </net>
+<net name="N$22" class="0">
+<segment>
+<pinref part="U$6" gate="G$1" pin="1"/>
+<pinref part="U3" gate="G$1" pin="EN"/>
+<wire x1="444.5" y1="-45.72" x2="447.04" y2="-45.72" width="0.1524" layer="91"/>
+</segment>
+</net>

Commit message: temp
Parts:
- removed R7: 0.0, derek:CRCW06030000Z0EA
Connections:
- removed net N$13: R7.2, U1.DRV
- net N$12: now also U1.DRV; no longer R7.1
Changed lines of the file:
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@@
 <part name="R2" library="derek" deviceset="CRCW121033R2FKEA" device="" value="33.2"/>
 <part name="Q1" library="derek" deviceset="IPD65R600C6" device=""/>
-<part name="R7" library="derek" deviceset="CRCW06030000Z0EA" device="" value="0.0"/>
 <part name="R8" library="derek" deviceset="CRCW1206698RFKEA" device="" value="698"/>
 <part name="R3" library="derek" deviceset="CRCW12064R70JNEA" device="" value="4.7"/>
@@
 <instance part="R2" gate="G$1" x="142.24" y="-7.62" rot="R270"/>
 <instance part="Q1" gate="G$1" x="139.7" y="-116.84"/>
-<instance part="R7" gate="G$1" x="121.92" y="-119.38"/>
 <instance part="R8" gate="G$1" x="78.74" y="-134.62"/>
 <instance part="R3" gate="G$1" x="38.1" y="-63.5" rot="R90"/>
@@
 <net name="N$12" class="0">
 <segment>
-<pinref part="R7" gate="G$1" pin="1"/>
 <pinref part="Q1" gate="G$1" pin="G"/>
-<wire x1="129.54" y1="-119.38" x2="134.62" y2="-119.38" width="0.1524" layer="91"/>
+<pinref part="U1" gate="G$1" pin="DRV"/>
+<wire x1="134.62" y1="-119.38" x2="96.52" y2="-119.38" width="0.1524" layer="91"/>
 </segment>
 </net>
@@
 </segment>
 </net>
-<net name="N$13" class="0">
-<segment>
-<pinref part="R7" gate="G$1" pin="2"/>
-<pinref part="U1" gate="G$1" pin="DRV"/>
-<wire x1="114.3" y1="-119.38" x2="96.52" y2="-119.38" width="0.1524" layer="91"/>
-</segment>
-</net>

Commit message: ordered
Parts:
- removed C3: 220µF, derek:UHE1V221MPD6
- removed U$1, U$4, U$5: TP-1502, derek:TP-1502
- removed U$6: 10k, derek:CRCW060310K0FKEA
- removed U3: ESP-WROOM-32, derek:ESP-WROOM-32
- C2: value 220µF -> 470µF; device derek:UHE1V221MPD6 -> derek:EEU-EB1V471
Connections:
- removed net N$21: U$1.TP, U3.IO25
- removed net N$22: U$6.1, U3.EN
- removed net N$23: U$5.TP, U3.IO27
- removed net N$24: U$4.TP, U3.IO26
- net 24V: no longer C3.1
- net 3.3V: no longer U$6.2, U3.3V3
- net GND-ISO: no longer C3.2, U3.GND, U3.GND@1, U3.GND@15, U3.GND@38
Changed lines of the file:
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@@
 <?xml version="1.0" encoding="utf-8"?>
 <!DOCTYPE eagle SYSTEM "eagle.dtd">
-<eagle version="8.2.0">
+<eagle version="8.2.2">
 <drawing>
 <settings>
@@
 <part name="C4" library="derek" deviceset="UMK316AB7475KL-T" device="" value="4.7µF"/>
 <part name="C5" library="derek" deviceset="UMK316AB7475KL-T" device="" value="4.7µF"/>
-<part name="C2" library="derek" deviceset="UHE1V221MPD6" device="" value="220µF"/>
-<part name="C3" library="derek" deviceset="UHE1V221MPD6" device="" value="220µF"/>
+<part name="C2" library="derek" deviceset="EEU-EB1V471" device="" value="470µF"/>
 <part name="C6" library="derek" deviceset="08053C104KAT2A" device="" value="0.1µF"/>
 <part name="R1" library="derek" deviceset="CRCW120610K0JNEA" device="" value="10k"/>
@@
 <part name="F1" library="derek" deviceset="37012000410" device=""/>
 <part name="GND25" library="derek" deviceset="GND" device=""/>
-<part name="U3" library="derek" deviceset="ESP-WROOM-32" device=""/>
-<part name="U$1" library="derek" deviceset="TP-1502" device=""/>
-<part name="U$4" library="derek" deviceset="TP-1502" device=""/>
-<part name="SUPPLY7" library="derek" deviceset="3.3V" device=""/>
-<part name="GND-ISO5" library="derek" deviceset="GND-ISO" device=""/>
-<part name="GND-ISO6" library="derek" deviceset="GND-ISO" device=""/>
-<part name="GND-ISO7" library="derek" deviceset="GND-ISO" device=""/>
-<part name="GND-ISO8" library="derek" deviceset="GND-ISO" device=""/>
-<part name="U$5" library="derek" deviceset="TP-1502" device=""/>
-<part name="U$6" library="derek" deviceset="CRCW060310K0FKEA" device="" value="10k"/>
 </parts>
 <sheets>
@@
 <instance part="C5" gate="G$1" x="241.3" y="35.56" rot="R90"/>
 <instance part="C2" gate="G$1" x="251.46" y="35.56" rot="R90"/>
-<instance part="C3" gate="G$1" x="264.16" y="35.56" rot="R90"/>
 <instance part="C6" gate="A" x="276.86" y="35.56" rot="R90"/>
 <instance part="R1" gate="G$1" x="287.02" y="35.56" rot="R90"/>
@@
 <instance part="F1" gate="G$1" x="48.26" y="25.4"/>
 <instance part="GND25" gate="G$1" x="55.88" y="-119.38"/>
-<instance part="U3" gate="G$1" x="464.82" y="-43.18"/>
-<instance part="U$1" gate="A" x="429.26" y="-53.34"/>
-<instance part="U$4" gate="A" x="429.26" y="-76.2"/>
-<instance part="SUPPLY7" gate="G$1" x="426.72" y="-40.64"/>
-<instance part="GND-ISO5" gate="G$1" x="434.34" y="-38.1"/>
-<instance part="GND-ISO6" gate="G$1" x="459.74" y="-93.98"/>
-<instance part="GND-ISO7" gate="G$1" x="508" y="-45.72"/>
-<instance part="GND-ISO8" gate="G$1" x="472.44" y="-68.58"/>
-<instance part="U$5" gate="A" x="429.26" y="-96.52"/>
-<instance part="U$6" gate="G$1" x="436.88" y="-45.72"/>
 </instances>
 <busses>
@@
 <junction x="467.36" y="33.02"/>
 </segment>
-<segment>
-<pinref part="U3" gate="G$1" pin="3V3"/>
-<pinref part="SUPPLY7" gate="G$1" pin="3.3V"/>
-<wire x1="447.04" y1="-43.18" x2="426.72" y2="-43.18" width="0.1524" layer="91"/>
-<wire x1="426.72" y1="-43.18" x2="426.72" y2="-40.64" width="0.1524" layer="91"/>
-<pinref part="U$6" gate="G$1" pin="2"/>
-<wire x1="429.26" y1="-45.72" x2="426.72" y2="-45.72" width="0.1524" layer="91"/>
-<wire x1="426.72" y1="-45.72" x2="426.72" y2="-43.18" width="0.1524" layer="91"/>
-<junction x="426.72" y="-43.18"/>
-</segment>
 </net>
 <net name="GND" class="0">
@@
 <wire x1="231.14" y1="25.4" x2="241.3" y2="25.4" width="0.1524" layer="91"/>
 <wire x1="241.3" y1="25.4" x2="251.46" y2="25.4" width="0.1524" layer="91"/>
-<wire x1="251.46" y1="25.4" x2="264.16" y2="25.4" width="0.1524" layer="91"/>
-<wire x1="264.16" y1="25.4" x2="276.86" y2="25.4" width="0.1524" layer="91"/>
+<wire x1="251.46" y1="25.4" x2="276.86" y2="25.4" width="0.1524" layer="91"/>
 <wire x1="276.86" y1="25.4" x2="287.02" y2="25.4" width="0.1524" layer="91"/>
 <wire x1="287.02" y1="25.4" x2="297.18" y2="25.4" width="0.1524" layer="91"/>
@@
 <wire x1="251.46" y1="27.94" x2="251.46" y2="25.4" width="0.1524" layer="91"/>
 <junction x="251.46" y="25.4"/>
-<pinref part="C3" gate="G$1" pin="2"/>
-<wire x1="264.16" y1="27.94" x2="264.16" y2="25.4" width="0.1524" layer="91"/>
-<junction x="264.16" y="25.4"/>
 <pinref part="C6" gate="A" pin="2"/>
 <wire x1="276.86" y1="27.94" x2="276.86" y2="25.4" width="0.1524" layer="91"/>
@@
 <wire x1="381" y1="45.72" x2="381" y2="48.26" width="0.1524" layer="91"/>
 </segment>
-<segment>
-<pinref part="U3" gate="G$1" pin="GND@1"/>
-<pinref part="GND-ISO5" gate="G$1" pin="GND-ISO"/>
-<wire x1="447.04" y1="-40.64" x2="444.5" y2="-40.64" width="0.1524" layer="91"/>
-<wire x1="444.5" y1="-40.64" x2="444.5" y2="-33.02" width="0.1524" layer="91"/>
-<wire x1="444.5" y1="-33.02" x2="434.34" y2="-33.02" width="0.1524" layer="91"/>
-<wire x1="434.34" y1="-33.02" x2="434.34" y2="-35.56" width="0.1524" layer="91"/>
-</segment>
-<segment>
-<pinref part="U3" gate="G$1" pin="GND@15"/>
-<pinref part="GND-ISO6" gate="G$1" pin="GND-ISO"/>
-<wire x1="459.74" y1="-83.82" x2="459.74" y2="-91.44" width="0.1524" layer="91"/>
-</segment>
-<segment>
-<pinref part="U3" gate="G$1" pin="GND@38"/>
-<pinref part="GND-ISO7" gate="G$1" pin="GND-ISO"/>
-<wire x1="495.3" y1="-40.64" x2="508" y2="-40.64" width="0.1524" layer="91"/>
-<wire x1="508" y1="-40.64" x2="508" y2="-43.18" width="0.1524" layer="91"/>
-</segment>
-<segment>
-<pinref part="U3" gate="G$1" pin="GND"/>
-<pinref part="GND-ISO8" gate="G$1" pin="GND-ISO"/>
-<wire x1="472.44" y1="-60.96" x2="472.44" y2="-66.04" width="0.1524" layer="91"/>
-</segment>
 </net>
 <net name="24V" class="0">
@@
 <wire x1="231.14" y1="45.72" x2="241.3" y2="45.72" width="0.1524" layer="91"/>
 <wire x1="241.3" y1="45.72" x2="251.46" y2="45.72" width="0.1524" layer="91"/>
-<wire x1="251.46" y1="45.72" x2="264.16" y2="45.72" width="0.1524" layer="91"/>
-<wire x1="264.16" y1="45.72" x2="276.86" y2="45.72" width="0.1524" layer="91"/>
+<wire x1="251.46" y1="45.72" x2="276.86" y2="45.72" width="0.1524" layer="91"/>
 <wire x1="276.86" y1="45.72" x2="287.02" y2="45.72" width="0.1524" layer="91"/>
 <wire x1="287.02" y1="45.72" x2="297.18" y2="45.72" width="0.1524" layer="91"/>
@@
 <wire x1="251.46" y1="43.18" x2="251.46" y2="45.72" width="0.1524" layer="91"/>
 <junction x="251.46" y="45.72"/>
-<pinref part="C3" gate="G$1" pin="1"/>
-<wire x1="264.16" y1="43.18" x2="264.16" y2="45.72" width="0.1524" layer="91"/>
-<junction x="264.16" y="45.72"/>
 <pinref part="C6" gate="A" pin="1"/>
 <wire x1="276.86" y1="43.18" x2="276.86" y2="45.72" width="0.1524" layer="91"/>
@@
 </segment>
 </net>
-<net name="N$23" class="0">
-<segment>
-<pinref part="U$5" gate="A" pin="TP"/>
-<wire x1="436.88" y1="-96.52" x2="429.26" y2="-96.52" width="0.1524" layer="91"/>
-<pinref part="U3" gate="G$1" pin="IO27"/>
-<wire x1="447.04" y1="-68.58" x2="436.88" y2="-68.58" width="0.1524" layer="91"/>
-<wire x1="436.88" y1="-68.58" x2="436.88" y2="-96.52" width="0.1524" layer="91"/>
-</segment>
-</net>
-<net name="N$24" class="0">
-<segment>
-<pinref part="U$4" gate="A" pin="TP"/>
-<wire x1="434.34" y1="-76.2" x2="429.26" y2="-76.2" width="0.1524" layer="91"/>
-<pinref part="U3" gate="G$1" pin="IO26"/>
-<wire x1="447.04" y1="-66.04" x2="434.34" y2="-66.04" width="0.1524" layer="91"/>
-<wire x1="434.34" y1="-66.04" x2="434.34" y2="-76.2" width="0.1524" layer="91"/>
-</segment>
-</net>
-<net name="N$21" class="0">
-<segment>
-<pinref part="U3" gate="G$1" pin="IO25"/>
-<wire x1="447.04" y1="-63.5" x2="434.34" y2="-63.5" width="0.1524" layer="91"/>
-<wire x1="434.34" y1="-63.5" x2="434.34" y2="-53.34" width="0.1524" layer="91"/>
-<pinref part="U$1" gate="A" pin="TP"/>
-<wire x1="434.34" y1="-53.34" x2="429.26" y2="-53.34" width="0.1524" layer="91"/>
-</segment>
-</net>
-<net name="N$22" class="0">
-<segment>
-<pinref part="U$6" gate="G$1" pin="1"/>
-<pinref part="U3" gate="G$1" pin="EN"/>
-<wire x1="444.5" y1="-45.72" x2="447.04" y2="-45.72" width="0.1524" layer="91"/>
-</segment>
-</net>

Commit message: save
Parts:
- C7: value 47µF -> EEU-ED2G470S; device derek:EEU-ED2G470 -> derek:EEU-ED2G470S
Changed lines of the file:
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@@
 <part name="U$2" library="derek" deviceset="TP-1502" device=""/>
 <part name="U$3" library="derek" deviceset="TP-1502" device=""/>
-<part name="C7" library="derek" deviceset="EEU-ED2G470" device="" value="47µF"/>
+<part name="C7" library="derek" deviceset="EEU-ED2G470S" device="" value="EEU-ED2G470S"/>
 <part name="U$9" library="derek" deviceset="TP-1502" device=""/>
 <part name="U$10" library="derek" deviceset="TP-1502" device=""/>

Commit message: ORDERED
Parts:
- removed C_1: 2.2µF, derek:C1608X5R1V225K080AC
- removed C_2: 22µF, derek:GRM21BR60J226ME39L
- removed L_1: 10µH, derek:SDR0503-100ML
- removed R101: 10k, derek:CRCW120610K0JNEA
- removed R_1: 100k, derek:CRCW0402100KFKED
- removed U$8: TP-1502, derek:TP-1502
- removed U_1: TPS62177, derek:TPS62177
- added 3.3V: TP-1502, derek:TP-1502
- added C10: 2.2µF, derek:C1608X5R1V225K080AC
- added C11: 22µF, derek:GRM21BR60J226ME39L
- added C3: EEU-ED2G470S, derek:EEU-ED2G470S
- added L1: 10µH, derek:SDR0503-100ML
- added R12: 100k, derek:CRCW0402100KFKED
- added R7: 33.2, derek:CRCW121033R2FKEA
- added U2: TPS62177, derek:TPS62177
- C1: value 2200pF -> 0.1µF; device derek:DE1E3KX222MA4BN01F -> derek:06035C104KAT2A
- C2: value 470µF -> 2.2µF; device derek:EEU-EB1V471 -> derek:GRM31CR61H225KA88L
- C4: value 4.7µF -> 2200pF; device derek:UMK316AB7475KL-T -> derek:DE1E3KX222MA4BN01F
- C6: value 0.1µF -> 4.7µF; device derek:08053C104KAT2A -> derek:UMK316AB7475KL-T
- C7: value EEU-ED2G470S -> 220µF; device derek:EEU-ED2G470S -> derek:UHE1V221MPD6
- C8: value 0.1µF -> 220µF; device derek:06035C104KAT2A -> derek:UHE1V221MPD6
- C9: value 2.2µF -> 0.1µF; device derek:GRM31CR61H225KA88L -> derek:08053C104KAT2A
- D1: value SK4200L-TP -> BAS20HT1G; device derek:SK4200L-TP -> derek:BAS20HT1G
- D2: value SMAJ120A -> RH06-T; device derek:SMAJ120A -> derek:RH06-T
- D3: value RH06-T -> SMAJ120A; device derek:RH06-T -> derek:SMAJ120A
- D5: value BAS20HT1G -> SK4200L-TP; device derek:BAS20HT1G -> derek:SK4200L-TP
- R1: value 10k -> 75k; device derek:CRCW120610K0JNEA -> derek:CRCW060375K0FKEA
- R10: value 0.75 -> 10k; device derek:CSR1206FKR750 -> derek:CRCW120610K0JNEA
- R11: value 19.6k -> 10k; device derek:CRCW060319K6FKEA -> derek:CRCW120610K0JNEA
- R2: value 33.2 -> 19.6k; device derek:CRCW121033R2FKEA -> derek:CRCW060319K6FKEA
- R4: value 75k -> 698; device derek:CRCW060375K0FKEA -> derek:CRCW1206698RFKEA
- R8: value 698 -> 0.75; device derek:CRCW1206698RFKEA -> derek:CSR1206FKR750
- renumbered U$10 to GND, U$2 to L, U$3 to N, U$9 to 24V
Connections:
- net 24V: now also C10.1, C7.1, C8.1, C9.1, D5.C, R10.1, R11.1, U2.EN, U2.VIN; no longer C2.1, C4.1, C_1.1, D1.C, R1.1, R101.1, U_1.EN, U_1.VIN
- net 3.3V: now also 3.3V.TP, C11.1, L1.2, R12.1, U2.SLEEP, U2.VOS; no longer C_2.1, L_1.2, R_1.1, U$8.TP, U_1.SLEEP, U_1.VOS
- net GND: now also C2.2, C3.2, C4.2, D2.P$2, R2.2, R8.2; no longer C7.2, C8.2, C9.2, D3.P$2, R10.2, R11.2
- net GND-ISO: now also C10.2, C11.2, C4.1, C7.2, C8.2, C9.2, R10.2, R11.2, U2.AGND, U2.FB, U2.NC, U2.PGND; no longer C1.1, C2.2, C4.2, C_1.2, C_2.2, R1.2, R101.2, U_1.AGND, U_1.FB, U_1.NC, U_1.PGND
- net N$1: now also D2.P$4; no longer D3.P$4
- net N$10: now also R7.1; no longer R2.1
- net N$14: now also C1.1, C2.1, D1.C; no longer C8.1, C9.1, D5.C
- net N$15: now also R4.1; no longer R10.1
- net N$16: now also D1.A; no longer D5.A
- net N$17: now also R1.1; no longer R4.1
- net N$18: now also R4.2; no longer R8.2
- net N$2: now also D2.P$3; no longer D3.P$3
- net N$20: now also R1.2, R2.1; no longer R11.1, R4.2
- net N$3: now also C3.1, D2.P$1, D3.A; no longer C7.1, D2.A, D3.P$1
- net N$4: now also R12.2, U2.PG; no longer R_1.2, U_1.PG
- net N$5: now also L1.1, U2.SW; no longer L_1.1, U_1.SW
- net N$6: now also D5.A; no longer D1.A
- net N$8: now also D3.C; no longer D2.C
- net N$9: now also R7.2; no longer R2.2
Other:
- moved on the sheet: C1, C4, C5, C7, R1, R10, R11, R2, R4, R8, R9

Commit message: use this
Parts:
- C3: value EEU-ED2G470S -> 47µF
Changed lines of the file:
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@@
 <part name="L" library="derek" deviceset="TP-1502" device=""/>
 <part name="N" library="derek" deviceset="TP-1502" device=""/>
-<part name="C3" library="derek" deviceset="EEU-ED2G470S" device="" value="EEU-ED2G470S"/>
+<part name="C3" library="derek" deviceset="EEU-ED2G470S" device="" value="47µF"/>
 <part name="24V" library="derek" deviceset="TP-1502" device=""/>
 <part name="GND" library="derek" deviceset="TP-1502" device=""/>
