File: ctrl.sch (EAGLE design)
At the start: 47 parts, among them U1 TPS92513, U2 TPS92513

Commit message: save
Parts:
- removed D10, D11, D12, D13, D14, D3, D4, D5, D6, D7: XPGWHT-L1-0000-00BE8, derek:XPGWHT-L1-0000-00BE8
- removed J45: (no value), derek:CONN_07NO_SILK
- added U$1, U$2: 10M, derek:CRCW040210M0JNED
- added U$10, U$3, U$4, U$5, U$7, U$8, U$9: TP-1502, derek:TP-1502
- added U$6: 10k, derek:CRCW060310K0FKEA
- added U3: ESP-WROOM-32, derek:ESP-WROOM-32
Connections:
- removed net N$12: D6.C, D7.A
- removed net N$13: D3.C, D4.A
- removed net N$14: D4.C, D5.A
- removed net N$15: D5.C, D6.A
- removed net N$2: D11.C, D12.A
- removed net N$22: D13.C, D14.A
- removed net N$24: D10.A, D14.C
- removed net N$27: D10.C, D11.A
- new net 3.3V: U$3.TP, U$6.2, U3.3V3
- new net N$29: U$6.1, U3.EN
- net 24V: now also U$1.2, U$2.2, U$4.TP; no longer J45.7
- net CLK: now also U3.IO25; no longer J45.1
- net GND-ISO: now also U$10.TP, U3.GND, U3.GND@1, U3.GND@15, U3.GND@38; no longer D10.GND, D11.GND, D12.GND, D13.GND, D14.GND, D3.GND, D4.GND, D5.GND, D6.GND, D7.GND, J45.6
- net IADJ1: now also U$1.1; no longer J45.5
- net IADJ2: now also U$2.1; no longer J45.2
- net N$23: now also U$8.TP; no longer D12.C
- net N$26: now also U$9.TP; no longer D13.A
- net N$6: now also U$7.TP; no longer D3.A
- net N$7: now also U$5.TP; no longer D7.C
- net PDIM1: now also U3.IO26; no longer J45.4
- net PDIM2: now also U3.IO27; no longer J45.3

Commit message: saveeee
Parts:
- renumbered U$10 to GND, U$3 to 3.3V, U$4 to 24V, U$5 to C+, U$7 to C-, U$8 to W+, U$9 to W-
Changed lines of the file:
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@@
 <part name="SUPPLY2" library="derek" deviceset="24V" device=""/>
 <part name="SUPPLY3" library="derek" deviceset="24V" device=""/>
-<part name="U$3" library="derek" deviceset="TP-1502" device=""/>
-<part name="U$4" library="derek" deviceset="TP-1502" device=""/>
-<part name="U$5" library="derek" deviceset="TP-1502" device=""/>
-<part name="U$7" library="derek" deviceset="TP-1502" device=""/>
-<part name="U$8" library="derek" deviceset="TP-1502" device=""/>
-<part name="U$9" library="derek" deviceset="TP-1502" device=""/>
-<part name="U$10" library="derek" deviceset="TP-1502" device=""/>
+<part name="3.3V" library="derek" deviceset="TP-1502" device=""/>
+<part name="24V" library="derek" deviceset="TP-1502" device=""/>
+<part name="C+" library="derek" deviceset="TP-1502" device=""/>
+<part name="C-" library="derek" deviceset="TP-1502" device=""/>
+<part name="W+" library="derek" deviceset="TP-1502" device=""/>
+<part name="W-" library="derek" deviceset="TP-1502" device=""/>
+<part name="GND" library="derek" deviceset="TP-1502" device=""/>
 </parts>
 <sheets>
@@
 <instance part="SUPPLY2" gate="G$1" x="-137.16" y="78.74"/>
 <instance part="SUPPLY3" gate="G$1" x="-137.16" y="68.58"/>
-<instance part="U$3" gate="A" x="-198.12" y="177.8"/>
-<instance part="U$4" gate="A" x="-152.4" y="76.2"/>
-<instance part="U$5" gate="A" x="88.9" y="167.64" rot="R180"/>
-<instance part="U$7" gate="A" x="88.9" y="142.24" rot="R180"/>
-<instance part="U$8" gate="A" x="91.44" y="45.72" rot="R180"/>
-<instance part="U$9" gate="A" x="91.44" y="20.32" rot="R180"/>
-<instance part="U$10" gate="A" x="-99.06" y="180.34" rot="R180"/>
+<instance part="3.3V" gate="A" x="-198.12" y="177.8"/>
+<instance part="24V" gate="A" x="-152.4" y="76.2"/>
+<instance part="C+" gate="A" x="88.9" y="167.64" rot="R180"/>
+<instance part="C-" gate="A" x="88.9" y="142.24" rot="R180"/>
+<instance part="W+" gate="A" x="91.44" y="45.72" rot="R180"/>
+<instance part="W-" gate="A" x="91.44" y="20.32" rot="R180"/>
+<instance part="GND" gate="A" x="-99.06" y="180.34" rot="R180"/>
 </instances>
 <busses>
@@
 <wire x1="73.66" y1="142.24" x2="88.9" y2="142.24" width="0.1524" layer="91"/>
 <junction x="73.66" y="142.24"/>
-<pinref part="U$7" gate="A" pin="TP"/>
+<pinref part="C-" gate="A" pin="TP"/>
 </segment>
 </net>
@@
 <wire x1="25.4" y1="177.8" x2="73.66" y2="177.8" width="0.1524" layer="91"/>
 <wire x1="73.66" y1="177.8" x2="73.66" y2="167.64" width="0.1524" layer="91"/>
-<pinref part="U$5" gate="A" pin="TP"/>
+<pinref part="C+" gate="A" pin="TP"/>
 <wire x1="88.9" y1="167.64" x2="73.66" y2="167.64" width="0.1524" layer="91"/>
 </segment>
@@
 <wire x1="-119.38" y1="180.34" x2="-106.68" y2="180.34" width="0.1524" layer="91"/>
 <wire x1="-106.68" y1="180.34" x2="-106.68" y2="177.8" width="0.1524" layer="91"/>
-<pinref part="U$10" gate="A" pin="TP"/>
+<pinref part="GND" gate="A" pin="TP"/>
 <wire x1="-99.06" y1="180.34" x2="-106.68" y2="180.34" width="0.1524" layer="91"/>
 <junction x="-106.68" y="180.34"/>
@@
 <pinref part="SUPPLY2" gate="G$1" pin="24V"/>
 <wire x1="-137.16" y1="76.2" x2="-137.16" y2="78.74" width="0.1524" layer="91"/>
-<pinref part="U$4" gate="A" pin="TP"/>
+<pinref part="24V" gate="A" pin="TP"/>
 <wire x1="-152.4" y1="76.2" x2="-137.16" y2="76.2" width="0.1524" layer="91"/>
 <junction x="-137.16" y="76.2"/>
@@
 <pinref part="L2" gate="G$1" pin="2"/>
 <wire x1="73.66" y1="45.72" x2="63.5" y2="45.72" width="0.1524" layer="91"/>
-<pinref part="U$8" gate="A" pin="TP"/>
+<pinref part="W+" gate="A" pin="TP"/>
 <wire x1="91.44" y1="45.72" x2="73.66" y2="45.72" width="0.1524" layer="91"/>
 </segment>
@@
 <junction x="73.66" y="20.32"/>
 <wire x1="73.66" y1="20.32" x2="73.66" y2="-7.62" width="0.1524" layer="91"/>
-<pinref part="U$9" gate="A" pin="TP"/>
+<pinref part="W-" gate="A" pin="TP"/>
 <wire x1="91.44" y1="20.32" x2="73.66" y2="20.32" width="0.1524" layer="91"/>
 </segment>
@@
 <wire x1="-187.96" y1="175.26" x2="-187.96" y2="177.8" width="0.1524" layer="91"/>
 <junction x="-187.96" y="177.8"/>
-<pinref part="U$3" gate="A" pin="TP"/>
+<pinref part="3.3V" gate="A" pin="TP"/>
 <wire x1="-198.12" y1="177.8" x2="-187.96" y2="177.8" width="0.1524" layer="91"/>
 </segment>

Commit message: rearrange positions
Parts:
- removed 24V, 3.3V, C+, C-, GND: TP-1502, derek:TP-1502
- removed C10: 10000pF, derek:GCM155R71H103KA55D
- removed C11: 0.01μF, derek:CC0805KRX7R9BB103
- removed C12: 0.1µF, derek:CC0805KRX7R8BB104
- removed C13: 0.1µF, derek:GRM188R71E104KA01D
- removed C14: 1µF, derek:GMK212B7105KG-T
- removed C15, C9: 1µF, derek:GRM31MR71H105KA88L
- removed C16: 470pF, derek:C0603X471K5RACTU
- removed D8, D9: PMEG6010CEH,115, derek:PMEG6010CEH,115
- removed L2: 33µH, derek:SRN6045-330M
- removed R10: 976, derek:CRCW0402976RFKED
- removed R11: 0.51, derek:CRM0805-FX-R510ELF
- removed R12: 4.02k, derek:CRCW06034K02FKEA
- removed R9: 162k, derek:CRCW0402162KFKED
- removed U$1, U$2: 10M, derek:CRCW040210M0JNED
- removed U$6: 10k, derek:CRCW060310K0FKEA
- removed U3: ESP-WROOM-32, derek:ESP-WROOM-32
- added TP1, TP2, TP3: TP-1502, derek:TP-1502
- R5: value 976 -> 10M; device derek:CRCW0402976RFKED -> derek:CRCW040210M0JNED
- R6: value 0.51 -> 976; device derek:CRM0805-FX-R510ELF -> derek:CRCW0402976RFKED
- R7: value 97.6k -> 0.51; device derek:CRCW040297K6FKED -> derek:CRM0805-FX-R510ELF
- R8: value 5.49k -> 10k; device derek:CRCW04025K49FKED -> derek:CRCW060310K0FKEA
- U2: value TPS92513 -> ESP-WROOM-32; device derek:TPS92513 -> derek:ESP-WROOM-32
- renumbered W+ to TP4, W- to TP5
Connections:
- removed net IADJ1: C5.1, U$1.1, U1.IADJ
- removed net N$1 (its old number): R7.2, R8.1, U2.UVLO
- removed net N$11: R5.2, U1.ISENSE
- removed net N$16 (its old number): C13.1, D9.C, L2.1, U2.PH
- removed net N$17 (its old number): R12.2, R9.1, U2.RT/CLK
- removed net N$18 (its old number): C12.1, U2.COMP
- removed net N$19 (its old number): C13.2, U2.BOOT
- removed net N$25 (its old number): C16.1, R12.1
- removed net N$6: C-.TP, C8.2, R5.1, R6.1
- removed net N$7: C+.TP, C8.1, D1.A, L1.2
- net 24V: now also R5.2, TP2.TP; no longer 24V.TP, C10.1, C15.1, C9.1, D8.C, R7.1, U$1.2, U$2.2, U2.VIN
- net 3.3V: now also R8.2, TP1.TP, U2.3V3; no longer 3.3V.TP, U$6.2, U3.3V3
- net CLK: now also U2.IO25; no longer C16.2, U3.IO25
- net GND-ISO: now also R7.2, TP3.TP, U2.GND@1, U2.GND@15, U2.GND@38; no longer C10.2, C11.2, C12.2, C15.2, C9.2, D9.A, GND.TP, R11.2, R6.2, R8.2, R9.2, U3.GND, U3.GND@1, U3.GND@15, U3.GND@38
- net IADJ2: now also C5.1, R5.1, U1.IADJ; no longer C11.1, U$2.1, U2.IADJ
- net N$20: now also R6.2, U1.ISENSE; no longer R10.2, U2.ISENSE
- net N$23: now also C8.1, D1.A, L1.2; no longer C14.1, D8.A, L2.2
- net N$26: now also C8.2, R6.1, R7.1; no longer C14.2, R10.1, R11.1
- net N$29: now also R8.1, U2.EN; no longer U$6.1, U3.EN
- net PDIM1: now also U2.IO26; no longer U1.PDIM, U3.IO26
- net PDIM2: now also U1.PDIM, U2.IO27; no longer U2.PDIM, U3.IO27
Other:
- moved on the sheet: C1, C2, C3, C4, C5, C6, C7, C8, D1, D2, L1, R1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

Commit message: save
Parts:
- added C+, C-: TP-1502, derek:TP-1502
- added C10, C9: 1µF, derek:GRM31MR71H105KA88L
- added C11: 10000pF, derek:GCM155R71H103KA55D
- added C12: 470pF, derek:C0603X471K5RACTU
- added C13: 0.01μF, derek:CC0805KRX7R9BB103
- added C14: 0.1µF, derek:GRM188R71E104KA01D
- added C15: 0.1µF, derek:CC0805KRX7R8BB104
- added C16: 1µF, derek:GMK212B7105KG-T
- added D3, D4: PMEG6010CEH,115, derek:PMEG6010CEH,115
- added L2: 33µH, derek:SRN6045-330M
- added R10: 162k, derek:CRCW0402162KFKED
- added R11: 4.02k, derek:CRCW06034K02FKEA
- added R12: 10M, derek:CRCW040210M0JNED
- added R13: 976, derek:CRCW0402976RFKED
- added R14: 0.51, derek:CRM0805-FX-R510ELF
- added R15: 10k, derek:CRCW060310K0FKEA
- added R9: 5.49k, derek:CRCW04025K49FKED
- added U3: ESP-WROOM-32, derek:ESP-WROOM-32
- R8: value 10k -> 97.6k; device derek:CRCW060310K0FKEA -> derek:CRCW040297K6FKED
- U2: value ESP-WROOM-32 -> TPS92513; device derek:ESP-WROOM-32 -> derek:TPS92513
- renumbered TP1 to 3.3V, TP2 to 24V, TP3 to GND, TP4 to W+, TP5 to W-
Connections:
- new net IADJ1: C13.1, R12.1, U2.IADJ
- new net N$10: C-.TP, C16.2, R13.1, R14.1
- new net N$2: R8.2, R9.1, U2.UVLO
- new net N$3: C14.1, D4.C, L2.1, U2.PH
- new net N$4: R10.1, R11.2, U2.RT/CLK
- new net N$5: C15.1, U2.COMP
- new net N$6: C14.2, U2.BOOT
- new net N$7: R13.2, U2.ISENSE
- new net N$8: C12.1, R11.1
- new net N$9: C+.TP, C16.1, D3.A, L2.2
- net 24V: now also C10.1, C11.1, C9.1, D3.C, R12.2, R8.1, U2.VIN
- net 3.3V: now also R15.2, U3.3V3; no longer R8.2, U2.3V3
- net CLK: now also C12.2, U3.IO25; no longer U2.IO25
- net GND-ISO: now also C10.2, C11.2, C13.2, C15.2, C9.2, D4.A, R10.2, R14.2, R9.2, U3.GND, U3.GND@1, U3.GND@15, U3.GND@38; no longer U2.GND@1, U2.GND@15, U2.GND@38
- net N$29: now also R15.1, U3.EN; no longer R8.1, U2.EN
- net PDIM1: now also U2.PDIM, U3.IO26; no longer U2.IO26
- net PDIM2: now also U3.IO27; no longer U2.IO27
Other:
- moved on the sheet: R8
